Commit message: Fixed the URDF for better readabilty

File: urdf/asv_base.urdf.xacro (robot description, xacro)
@@ -1,5 +1,11 @@
 <?xml version="1.0"?>
 <robot xmlns:xacro="http://www.ros.org/wiki/xacro" name="asv_description">
-  <link name="asv">
+  <gazebo>
+    <plugin name="ros_control" filename="libgazebo_ros_control.so">
+      <robotNamespace>/boat</robotNamespace>
+      <robotSimType>gazebo_ros_control/DefaultRobotHWSim</robotSimType>
+    </plugin>
+  </gazebo>
+   <link name="base_footprint">
     <inertial>
       <origin rpy="0 0 0" xyz="0.38789 0.59329 1.1865"/>
@@ -47,5 +53,5 @@
   <joint name="body_to_thruster_right" type="fixed">
     <origin rpy="1.5708 0 3.1416" xyz="0.74762 -1.335 0.37124"/>
-    <parent link="asv"/>
+    <parent link="base_footprint"/>
     <child link="thruster_right"/>
     <axis xyz="0 0 0"/>
@@ -75,5 +81,5 @@
   <joint name="body_to_thruster_left" type="fixed">
     <origin rpy="1.5708 0 3.1416" xyz="0.027678 -1.335 0.37124"/>
-    <parent link="asv"/>
+    <parent link="base_footprint"/>
     <child link="thruster_left"/>
     <axis xyz="0 0 0"/>
@@ -103,5 +109,5 @@
   <joint name="asv_to_top_body" type="fixed">
     <origin rpy="1.5708 0 0" xyz="0.38708 -1.0625 0.60681"/>
-    <parent link="asv"/>
+    <parent link="base_footprint"/>
     <child link="top_body"/>
     <axis xyz="0 0 0"/>
@@ -356,5 +362,5 @@
   <joint name="body_to_battery" type="fixed">
     <origin rpy="3.1416 0 0" xyz="0.38768 -1.5211 0.59834"/>
-    <parent link="asv"/>
+    <parent link="base_footprint"/>
     <child link="battery_1"/>
     <axis xyz="0 0 0"/>
@@ -412,5 +418,5 @@
   <joint name="body_to_mount" type="fixed">
     <origin rpy="1.5708 0 0" xyz="0.38768 -1.2531 0.56334"/>
-    <parent link="asv"/>
+    <parent link="base_footprint"/>
     <child link="mount"/>
     <axis xyz="0 0 0"/>
@@ -472,3 +478,24 @@
     <axis xyz="0 0 0"/>
   </joint>
+  <gazebo reference="base_footprint">
+    <turnGravityOff>true</turnGravityOff>
+  </gazebo>
+  <gazebo reference="thruster_right">
+    <turnGravityOff>true</turnGravityOff>
+  </gazebo>
+  <gazebo reference="thruster_left">
+    <turnGravityOff>true</turnGravityOff>
+  </gazebo>
+  <gazebo reference="top_body">
+    <turnGravityOff>true</turnGravityOff>
+  </gazebo>
+    <gazebo reference="">
+    <turnGravityOff>true</turnGravityOff>
+  </gazebo>
+    <gazebo reference="">
+    <turnGravityOff>true</turnGravityOff>
+  </gazebo>
+    <gazebo reference="">
+    <turnGravityOff>true</turnGravityOff>
+  </gazebo>
 </robot>

Commit message: Integrated the ROS control transmissions to the ASV URDF

File: urdf/asv_base.urdf.xacro (robot description, xacro)
@@ -3,8 +3,9 @@
   <gazebo>
     <plugin name="ros_control" filename="libgazebo_ros_control.so">
-      <robotNamespace>/boat</robotNamespace>
+      <robotNamespace>/asv</robotNamespace>
       <robotSimType>gazebo_ros_control/DefaultRobotHWSim</robotSimType>
     </plugin>
   </gazebo>
+  <xacro:property name="PI" value="3.14159265359" />
    <link name="base_footprint">
     <inertial>
@@ -51,9 +52,11 @@
     </collision>
   </link>
-  <joint name="body_to_thruster_right" type="fixed">
+  <joint name="body_to_thruster_right" type="continuous">
     <origin rpy="1.5708 0 3.1416" xyz="0.74762 -1.335 0.37124"/>
     <parent link="base_footprint"/>
     <child link="thruster_right"/>
-    <axis xyz="0 0 0"/>
+    <axis xyz="0 1 0"/>
+       <limit effort="30" velocity="1.0" lower="-32000" upper="32000" />
+    <dynamics damping="0.1" friction="0.1" />
   </joint>
   <link name="thruster_left">
@@ -79,9 +82,11 @@
     </collision>
   </link>
-  <joint name="body_to_thruster_left" type="fixed">
+  <joint name="body_to_thruster_left" type="continuous">
     <origin rpy="1.5708 0 3.1416" xyz="0.027678 -1.335 0.37124"/>
     <parent link="base_footprint"/>
     <child link="thruster_left"/>
-    <axis xyz="0 0 0"/>
+    <axis xyz="0 1 0"/>
+       <limit effort="30" velocity="1.0" lower="-32000" upper="32000" />
+    <dynamics damping="0.1" friction="0.1" />
   </joint>
   <link name="top_body">
@@ -478,4 +483,22 @@
     <axis xyz="0 0 0"/>
   </joint>
+<transmission name="left_thruster_rotation">
+  <type>transmission_interface/SimpleTransmission</type>
+  <joint name="body_to_thruster_left">
+    <hardwareInterface>VelocityJointInterface</hardwareInterface>
+  </joint>
+  <actuator name="left_thruster_actuator">
+    <mechanicalReduction>1</mechanicalReduction>
+  </actuator>
+</transmission>
+<transmission name="right_thruster_rotation">
+  <type>transmission_interface/SimpleTransmission</type>
+  <joint name="body_to_thruster_right">
+    <hardwareInterface>VelocityJointInterface</hardwareInterface>
+  </joint>
+  <actuator name="right_thruster_actuator">
+    <mechanicalReduction>1</mechanicalReduction>
+  </actuator>
+</transmission>
   <gazebo reference="base_footprint">
     <turnGravityOff>true</turnGravityOff>
@@ -490,11 +513,41 @@
     <turnGravityOff>true</turnGravityOff>
   </gazebo>
-    <gazebo reference="">
-    <turnGravityOff>true</turnGravityOff>
-  </gazebo>
-    <gazebo reference="">
-    <turnGravityOff>true</turnGravityOff>
-  </gazebo>
-    <gazebo reference="">
+    <gazebo reference="top_cover">
+    <turnGravityOff>true</turnGravityOff>
+  </gazebo>
+    <gazebo reference="sensor_pod">
+    <turnGravityOff>true</turnGravityOff>
+  </gazebo>
+    <gazebo reference="camera_garmin_mounts">
+    <turnGravityOff>true</turnGravityOff>
+  </gazebo>
+    <gazebo reference="garmin">
+    <turnGravityOff>true</turnGravityOff>
+  </gazebo>
+    <gazebo reference="camera">
+    <turnGravityOff>true</turnGravityOff>
+  </gazebo>
+    <gazebo reference="lidar">
+    <turnGravityOff>true</turnGravityOff>
+  </gazebo>
+    <gazebo reference="kill_switch_1">
+    <turnGravityOff>true</turnGravityOff>
+  </gazebo>
+    <gazebo reference="kill_switch_2">
+    <turnGravityOff>true</turnGravityOff>
+  </gazebo>
+    <gazebo reference="battery_1">
+    <turnGravityOff>true</turnGravityOff>
+  </gazebo>
+    <gazebo reference="battery_2">
+    <turnGravityOff>true</turnGravityOff>
+  </gazebo>
+    <gazebo reference="mount">
+    <turnGravityOff>true</turnGravityOff>
+  </gazebo>
+    <gazebo reference="rs_232_port">
+    <turnGravityOff>true</turnGravityOff>
+  </gazebo>
+    <gazebo reference="status_board">
     <turnGravityOff>true</turnGravityOff>
   </gazebo>

Commit message: Xacro to replace path of model files

File: urdf/asv_base.urdf.xacro (robot description, xacro)
@@ -8,4 +8,5 @@
   </gazebo>
   <xacro:property name="PI" value="3.14159265359" />
+  <xacro:arg name="path" default="package://asv_description/meshes" />
    <link name="base_footprint">
     <inertial>
@@ -17,14 +18,14 @@
       <origin rpy="0 0 0" xyz="0 0 0"/>
       <geometry>
-        <mesh filename="package://asv_description/meshes/asv.STL"/>
-      </geometry>
-      <material name="">
-        <color rgba="0.79216 0.81961 0.93333 1"/>
-      </material>
-    </visual>
-    <collision>
-      <origin rpy="0 0 0" xyz="0 0 0"/>
-      <geometry>
-        <mesh filename="package://asv_description/meshes/asv.STL"/>
+        <mesh filename="$(arg path)/asv.STL"/>
+      </geometry>
+      <material name="">
+        <color rgba="0.79216 0.81961 0.93333 1"/>
+      </material>
+    </visual>
+    <collision>
+      <origin rpy="0 0 0" xyz="0 0 0"/>
+      <geometry>
+        <mesh filename="$(arg path)/asv.STL"/>
       </geometry>
     </collision>
@@ -39,14 +40,14 @@
       <origin rpy="0 0 0" xyz="0 0 0"/>
       <geometry>
-        <mesh filename="package://asv_description/meshes/thruster_right.STL"/>
-      </geometry>
-      <material name="">
-        <color rgba="0.79216 0.81961 0.93333 1"/>
-      </material>
-    </visual>
-    <collision>
-      <origin rpy="0 0 0" xyz="0 0 0"/>
-      <geometry>
-        <mesh filename="package://asv_description/meshes/thruster_right.STL"/>
+        <mesh filename="$(arg path)/thruster_right.STL"/>
+      </geometry>
+      <material name="">
+        <color rgba="0.79216 0.81961 0.93333 1"/>
+      </material>
+    </visual>
+    <collision>
+      <origin rpy="0 0 0" xyz="0 0 0"/>
+      <geometry>
+        <mesh filename="$(arg path)/thruster_right.STL"/>
       </geometry>
     </collision>
@@ -69,14 +70,14 @@
       <origin rpy="0 0 0" xyz="0 0 0"/>
       <geometry>
-        <mesh filename="package://asv_description/meshes/thruster_left.STL"/>
-      </geometry>
-      <material name="">
-        <color rgba="0.79216 0.81961 0.93333 1"/>
-      </material>
-    </visual>
-    <collision>
-      <origin rpy="0 0 0" xyz="0 0 0"/>
-      <geometry>
-        <mesh filename="package://asv_description/meshes/thruster_left.STL"/>
+        <mesh filename="$(arg path)/thruster_left.STL"/>
+      </geometry>
+      <material name="">
+        <color rgba="0.79216 0.81961 0.93333 1"/>
+      </material>
+    </visual>
+    <collision>
+      <origin rpy="0 0 0" xyz="0 0 0"/>
+      <geometry>
+        <mesh filename="$(arg path)/thruster_left.STL"/>
       </geometry>
     </collision>
@@ -99,5 +100,5 @@
       <origin rpy="0 0 0" xyz="0 0 0"/>
       <geometry>
-        <mesh filename="package://asv_description/meshes/top_body.STL"/>
+        <mesh filename="$(arg path)/top_body.STL"/>
       </geometry>
       <material name="">
@@ -108,5 +109,5 @@
       <origin rpy="0 0 0" xyz="0 0 0"/>
       <geometry>
-        <mesh filename="package://asv_description/meshes/top_body.STL"/>
+        <mesh filename="$(arg path)/top_body.STL"/>
       </geometry>
     </collision>
@@ -127,5 +128,5 @@
       <origin xyz="0 0 0" rpy="0 0 0" />
       <geometry>
-        <mesh filename="package://asv_description/meshes/top_cover.STL" />
+        <mesh filename="$(arg path)/top_cover.STL" />
       </geometry>
       <material name="">
@@ -136,5 +137,5 @@
       <origin xyz="0 0 0" rpy="0 0 0" />
       <geometry>
-        <mesh filename="package://asv_description/meshes/top_cover.STL" />
+        <mesh filename="$(arg path)/top_cover.STL" />
       </geometry>
     </collision>
@@ -156,14 +157,14 @@
       <origin rpy="0 0 0" xyz="0 0 0"/>
       <geometry>
-        <mesh filename="package://asv_description/meshes/sensor_pod.STL"/>
-      </geometry>
-      <material name="">
-        <color rgba="0.79216 0.81961 0.93333 1"/>
-      </material>
-    </visual>
-    <collision>
-      <origin rpy="0 0 0" xyz="0 0 0"/>
-      <geometry>
-        <mesh filename="package://asv_description/meshes/sensor_pod.STL"/>
+        <mesh filename="$(arg path)/sensor_pod.STL"/>
+      </geometry>
+      <material name="">
+        <color rgba="0.79216 0.81961 0.93333 1"/>
+      </material>
+    </visual>
+    <collision>
+      <origin rpy="0 0 0" xyz="0 0 0"/>
+      <geometry>
+        <mesh filename="$(arg path)/sensor_pod.STL"/>
       </geometry>
     </collision>
@@ -184,14 +185,14 @@
       <origin rpy="0 0 0" xyz="0 0 0"/>
       <geometry>
-        <mesh filename="package://asv_description/meshes/camera_garmin_mounts.STL"/>
-      </geometry>
-      <material name="">
-        <color rgba="0.79216 0.81961 0.93333 1"/>
-      </material>
-    </visual>
-    <collision>
-      <origin rpy="0 0 0" xyz="0 0 0"/>
-      <geometry>
-        <mesh filename="package://asv_description/meshes/camera_garmin_mounts.STL"/>
+        <mesh filename="$(arg path)/camera_garmin_mounts.STL"/>
+      </geometry>
+      <material name="">
+        <color rgba="0.79216 0.81961 0.93333 1"/>
+      </material>
+    </visual>
+    <collision>
+      <origin rpy="0 0 0" xyz="0 0 0"/>
+      <geometry>
+        <mesh filename="$(arg path)/camera_garmin_mounts.STL"/>
       </geometry>
     </collision>
@@ -212,5 +213,5 @@
       <origin rpy="3.141592653589793 0 0" xyz="0 0 0"/>
       <geometry>
-        <mesh filename="package://asv_description/meshes/garmin.STL"/>
+        <mesh filename="$(arg path)/garmin.STL"/>
       </geometry>
       <material name="">
@@ -221,5 +222,5 @@
       <origin rpy="3.141592653589793 0 0" xyz="0 0 0"/>
       <geometry>
-        <mesh filename="package://asv_description/meshes/garmin.STL"/>
+        <mesh filename="$(arg path)/garmin.STL"/>
       </geometry>
     </collision>
@@ -240,5 +241,5 @@
       <origin rpy="0 0 0" xyz="0 0 0"/>
       <geometry>
-        <mesh filename="package://asv_description/meshes/camera.STL"/>
+        <mesh filename="$(arg path)/camera.STL"/>
       </geometry>
       <material name="">
@@ -249,5 +250,5 @@
       <origin rpy="0 0 0" xyz="0 0 0"/>
       <geometry>
-        <mesh filename="package://asv_description/meshes/camera.STL"/>
+        <mesh filename="$(arg path)/camera.STL"/>
       </geometry>
     </collision>
@@ -268,14 +269,14 @@
       <origin rpy="0 0 0" xyz="0 0 0"/>
       <geometry>
-        <mesh filename="package://asv_description/meshes/lidar.STL"/>
-      </geometry>
-      <material name="">
-        <color rgba="0.79216 0.81961 0.93333 1"/>
-      </material>
-    </visual>
-    <collision>
-      <origin rpy="0 0 0" xyz="0 0 0"/>
-      <geometry>
-        <mesh filename="package://asv_description/meshes/lidar.STL"/>
+        <mesh filename="$(arg path)/lidar.STL"/>
+      </geometry>
+      <material name="">
+        <color rgba="0.79216 0.81961 0.93333 1"/>
+      </material>
+    </visual>
+    <collision>
+      <origin rpy="0 0 0" xyz="0 0 0"/>
+      <geometry>
+        <mesh filename="$(arg path)/lidar.STL"/>
       </geometry>
     </collision>
@@ -296,14 +297,14 @@
       <origin rpy="0 0 0" xyz="0 0 0"/>
       <geometry>
-        <mesh filename="package://asv_description/meshes/kill_switch_2.STL"/>
-      </geometry>
-      <material name="">
-        <color rgba="0.79216 0.81961 0.93333 1"/>
-      </material>
-    </visual>
-    <collision>
-      <origin rpy="0 0 0" xyz="0 0 0"/>
-      <geometry>
-        <mesh filename="package://asv_description/meshes/kill_switch_2.STL"/>
+        <mesh filename="$(arg path)/kill_switch_2.STL"/>
+      </geometry>
+      <material name="">
+        <color rgba="0.79216 0.81961 0.93333 1"/>
+      </material>
+    </visual>
+    <collision>
+      <origin rpy="0 0 0" xyz="0 0 0"/>
+      <geometry>
+        <mesh filename="$(arg path)/kill_switch_2.STL"/>
       </geometry>
     </collision>
@@ -324,14 +325,14 @@
       <origin rpy="0 0 0" xyz="0 0 0"/>
       <geometry>
-        <mesh filename="package://asv_description/meshes/kill_switch_1.STL"/>
-      </geometry>
-      <material name="">
-        <color rgba="0.79216 0.81961 0.93333 1"/>
-      </material>
-    </visual>
-    <collision>
-      <origin rpy="0 0 0" xyz="0 0 0"/>
-      <geometry>
-        <mesh filename="package://asv_description/meshes/kill_switch_1.STL"/>
+        <mesh filename="$(arg path)/kill_switch_1.STL"/>
+      </geometry>
+      <material name="">
+        <color rgba="0.79216 0.81961 0.93333 1"/>
+      </material>
+    </visual>
+    <collision>
+      <origin rpy="0 0 0" xyz="0 0 0"/>
+      <geometry>
+        <mesh filename="$(arg path)/kill_switch_1.STL"/>
       </geometry>
     </collision>
@@ -352,14 +353,14 @@
       <origin rpy="0 0 0" xyz="0 0 0"/>
       <geometry>
-        <mesh filename="package://asv_description/meshes/battery_1.STL"/>
-      </geometry>
-      <material name="">
-        <color rgba="0.79216 0.81961 0.93333 1"/>
-      </material>
-    </visual>
-    <collision>
-      <origin rpy="0 0 0" xyz="0 0 0"/>
-      <geometry>
-        <mesh filename="package://asv_description/meshes/battery_1.STL"/>
+        <mesh filename="$(arg path)/battery_1.STL"/>
+      </geometry>
+      <material name="">
+        <color rgba="0.79216 0.81961 0.93333 1"/>
+      </material>
+    </visual>
+    <collision>
+      <origin rpy="0 0 0" xyz="0 0 0"/>
+      <geometry>
+        <mesh filename="$(arg path)/battery_1.STL"/>
       </geometry>
     </collision>
@@ -380,14 +381,14 @@
       <origin rpy="0 0 0" xyz="0 0 0"/>
       <geometry>
-        <mesh filename="package://asv_description/meshes/battery_2.STL"/>
-      </geometry>
-      <material name="">
-        <color rgba="0.79216 0.81961 0.93333 1"/>
-      </material>
-    </visual>
-    <collision>
-      <origin rpy="0 0 0" xyz="0 0 0"/>
-      <geometry>
-        <mesh filename="package://asv_description/meshes/battery_2.STL"/>
+        <mesh filename="$(arg path)/battery_2.STL"/>
+      </geometry>
+      <material name="">
+        <color rgba="0.79216 0.81961 0.93333 1"/>
+      </material>
+    </visual>
+    <collision>
+      <origin rpy="0 0 0" xyz="0 0 0"/>
+      <geometry>
+        <mesh filename="$(arg path)/battery_2.STL"/>
       </geometry>
     </collision>
@@ -408,14 +409,14 @@
       <origin rpy="0 0 0" xyz="0 0 0"/>
       <geometry>
-        <mesh filename="package://asv_description/meshes/mount.STL"/>
-      </geometry>
-      <material name="">
-        <color rgba="0.79216 0.81961 0.93333 1"/>
-      </material>
-    </visual>
-    <collision>
-      <origin rpy="0 0 0" xyz="0 0 0"/>
-      <geometry>
-        <mesh filename="package://asv_description/meshes/mount.STL"/>
+        <mesh filename="$(arg path)/mount.STL"/>
+      </geometry>
+      <material name="">
+        <color rgba="0.79216 0.81961 0.93333 1"/>
+      </material>
+    </visual>
+    <collision>
+      <origin rpy="0 0 0" xyz="0 0 0"/>
+      <geometry>
+        <mesh filename="$(arg path)/mount.STL"/>
       </geometry>
     </collision>
@@ -436,14 +437,14 @@
       <origin rpy="0 0 0" xyz="0 0 0"/>
       <geometry>
-        <mesh filename="package://asv_description/meshes/rs_232_port.STL"/>
-      </geometry>
-      <material name="">
-        <color rgba="0.79216 0.81961 0.93333 1"/>
-      </material>
-    </visual>
-    <collision>
-      <origin rpy="0 0 0" xyz="0 0 0"/>
-      <geometry>
-        <mesh filename="package://asv_description/meshes/rs_232_port.STL"/>
+        <mesh filename="$(arg path)/rs_232_port.STL"/>
+      </geometry>
+      <material name="">
+        <color rgba="0.79216 0.81961 0.93333 1"/>
+      </material>
+    </visual>
+    <collision>
+      <origin rpy="0 0 0" xyz="0 0 0"/>
+      <geometry>
+        <mesh filename="$(arg path)/rs_232_port.STL"/>
       </geometry>
     </collision>
@@ -464,14 +465,14 @@
       <origin rpy="0 0 0" xyz="0 0 0"/>
       <geometry>
-        <mesh filename="package://asv_description/meshes/status_board.STL"/>
-      </geometry>
-      <material name="">
-        <color rgba="0.79216 0.81961 0.93333 1"/>
-      </material>
-    </visual>
-    <collision>
-      <origin rpy="0 0 0" xyz="0 0 0"/>
-      <geometry>
-        <mesh filename="package://asv_description/meshes/status_board.STL"/>
+        <mesh filename="$(arg path)/status_board.STL"/>
+      </geometry>
+      <material name="">
+        <color rgba="0.79216 0.81961 0.93333 1"/>
+      </material>
+    </visual>
+    <collision>
+      <origin rpy="0 0 0" xyz="0 0 0"/>
+      <geometry>
+        <mesh filename="$(arg path)/status_board.STL"/>
       </geometry>
     </collision>

Commit message: Fixed the Joints configuration file and included controllers in launch file

File: urdf/asv_base.urdf.xacro (robot description, xacro)
@@ -484,11 +484,20 @@
     <axis xyz="0 0 0"/>
   </joint>
+  <sensor name="lidar" update_rate="30">
+    <parent link="lidar" />
+    <origin xyz="0 0 0" rpy="0 0 0 " />
+    <ray>
+      <horizontal samples="100" resolution="1" min_angle="-1.5708" max_angle="1.5708" />
+      <vertical samples="1" resolution="1" min_angle="0" max_angle="0"/>
+    </ray>
+  </sensor>
 <transmission name="left_thruster_rotation">
   <type>transmission_interface/SimpleTransmission</type>
   <joint name="body_to_thruster_left">
-    <hardwareInterface>VelocityJointInterface</hardwareInterface>
+    <hardwareInterface>EffortJointInterface</hardwareInterface>
   </joint>
   <actuator name="left_thruster_actuator">
     <mechanicalReduction>1</mechanicalReduction>
+    <hardwareInterface>EffortJointInterface</hardwareInterface>
   </actuator>
 </transmission>
@@ -496,8 +505,9 @@
   <type>transmission_interface/SimpleTransmission</type>
   <joint name="body_to_thruster_right">
-    <hardwareInterface>VelocityJointInterface</hardwareInterface>
+    <hardwareInterface>EffortJointInterface</hardwareInterface>
   </joint>
   <actuator name="right_thruster_actuator">
     <mechanicalReduction>1</mechanicalReduction>
+    <hardwareInterface>EffortJointInterface</hardwareInterface>
   </actuator>
 </transmission>
