Commit message: The controls have been made. However, need another commit to make the thrusters to rotate on a perfect axis

File: urdf/asv_base.urdf.xacro (robot description, xacro)
@@ -12,5 +12,5 @@
     <inertial>
       <origin rpy="0 0 0" xyz="0.38789 0.59329 1.1865"/>
-      <mass value="0.5331"/>
+      <mass value="2.331"/>
       <inertia ixx="0" ixy="0" ixz="0" iyy="0" iyz="0" izz="0"/>
     </inertial>
@@ -57,5 +57,5 @@
     <parent link="base_footprint"/>
     <child link="thruster_right"/>
-    <axis xyz="0 1 0"/>
+    <axis xyz="0 -1 0"/>
        <limit effort="30" velocity="1.0" lower="-32000" upper="32000" />
     <dynamics damping="0.1" friction="0.1" />
@@ -151,5 +151,5 @@
     <inertial>
       <origin rpy="0 0 0" xyz="-0.029193 -0.040604 -0.010551"/>
-      <mass value="0.6495"/>
+      <mass value="0.06495"/>
       <inertia ixx="0.0016814" ixy="-1.4742E-07" ixz="-3.6677E-05" iyy="0.0016822" iyz="-6.7581E-06" izz="8.2722E-07"/>
     </inertial>
@@ -179,5 +179,5 @@
     <inertial>
       <origin rpy="0 0 0" xyz="0.0027436 0.024777 0.009305"/>
-      <mass value="0.11757"/>
+      <mass value="0.011757"/>
       <inertia ixx="0.0001482" ixy="1.0861E-19" ixz="-3.2822E-19" iyy="0.00013357" iyz="4.4199E-05" izz="1.4626E-05"/>
     </inertial>
@@ -207,5 +207,5 @@
     <inertial>
       <origin rpy="3.141592653589793 0 0" xyz="0 0.023342 0"/>
-      <mass value="0.3356"/>
+      <mass value="0.03356"/>
       <inertia ixx="0" ixy="0" ixz="0" iyy="0" iyz="0" izz="0"/>
     </inertial>
@@ -235,5 +235,5 @@
     <inertial>
       <origin rpy="0 0 0" xyz="-2.8934E-05 -0.010178 0.021487"/>
-      <mass value="0.041091"/>
+      <mass value="0.0041091"/>
       <inertia ixx="1.4847E-05" ixy="-3.2519E-08" ixz="-1.1631E-08" iyy="3.365E-06" iyz="-4.1204E-06" izz="1.1483E-05"/>
     </inertial>
@@ -291,5 +291,5 @@
     <inertial>
       <origin rpy="0 0 0" xyz="0.21906 0.04363 0.013308"/>
-      <mass value="0.048397"/>
+      <mass value="0.0048397"/>
       <inertia ixx="0" ixy="0" ixz="0" iyy="0" iyz="0" izz="0"/>
     </inertial>
@@ -319,5 +319,5 @@
     <inertial>
       <origin rpy="0 0 0" xyz="0.21906 0.04363 0.013308"/>
-      <mass value="0.048397"/>
+      <mass value="0.0048397"/>
       <inertia ixx="0" ixy="0" ixz="0" iyy="0" iyz="0" izz="0"/>
     </inertial>
@@ -495,9 +495,8 @@
   <type>transmission_interface/SimpleTransmission</type>
   <joint name="body_to_thruster_left">
-    <hardwareInterface>hardware_interface/VelocityJointInterface</hardwareInterface>
+    <hardwareInterface>hardware_interface/EffortJointInterface</hardwareInterface>
   </joint>
   <actuator name="left_thruster_actuator">
     <mechanicalReduction>1</mechanicalReduction>
-    <hardwareInterface>VelocityJointInterface</hardwareInterface>
   </actuator>
 </transmission>
@@ -505,9 +504,8 @@
   <type>transmission_interface/SimpleTransmission</type>
   <joint name="body_to_thruster_right">
-    <hardwareInterface>hardware_interface/VelocityJointInterface</hardwareInterface>
+    <hardwareInterface>hardware_interface/EffortJointInterface</hardwareInterface>
   </joint>
   <actuator name="right_thruster_actuator">
     <mechanicalReduction>1</mechanicalReduction>
-    <hardwareInterface>VelocityJointInterface</hardwareInterface>
   </actuator>
 </transmission>

Commit message: Right thruster built for controllers

File: urdf/asv_base.urdf.xacro (robot description, xacro)
@@ -24,12 +24,6 @@
       </material>
     </visual>
-    <collision>
-      <origin rpy="0 0 0" xyz="0 0 0"/>
-      <geometry>
-        <mesh filename="$(arg path)/asv.STL"/>
-      </geometry>
-    </collision>
-  </link>
-  <link name="thruster_right">
+  </link>
+  <link name="thruster_right_dummy">
     <inertial>
       <origin rpy="0 0 0" xyz="-4.8522E-05 0.00051157 0.0095278"/>
@@ -37,6 +31,18 @@
       <inertia ixx="9.1096E-05" ixy="3.0619E-09" ixz="-1.6688E-07" iyy="9.0558E-05" iyz="1.2699E-06" izz="1.246E-06"/>
     </inertial>
-    <visual>
-      <origin rpy="0 0 0" xyz="0 0 0"/>
+  </link>
+  <joint name="thruster_right_fix" type="fixed">
+    <origin xyz="0 -0.95 1.7088" rpy="1.5708 0 0" />
+    <parent link="base_footprint"/>
+    <child link="thruster_right_dummy"/>
+  </joint>
+  <link name="thruster_right">
+    <inertial>
+      <origin rpy="0 0 0" xyz="-4.8522E-05 0.00051157 0.0095278"/>
+      <mass value="0.2183"/>
+      <inertia ixx="9.1096E-05" ixy="3.0619E-09" ixz="-1.6688E-07" iyy="9.0558E-05" iyz="1.2699E-06" izz="1.246E-06"/>
+    </inertial>
+    <visual>
+      <origin rpy="0 1.5708 1.5708" xyz="0 0 0"/>
       <geometry>
         <mesh filename="$(arg path)/thruster_right.STL"/>
@@ -46,14 +52,8 @@
       </material>
     </visual>
-    <collision>
-      <origin rpy="0 0 0" xyz="0 0 0"/>
-      <geometry>
-        <mesh filename="$(arg path)/thruster_right.STL"/>
-      </geometry>
-    </collision>
   </link>
   <joint name="body_to_thruster_right" type="continuous">
     <origin rpy="1.5708 0 3.1416" xyz="0.74762 -1.335 0.37124"/>
-    <parent link="base_footprint"/>
+    <parent link="thruster_right_dummy"/>
     <child link="thruster_right"/>
     <axis xyz="0 -1 0"/>
@@ -516,4 +516,7 @@
     <turnGravityOff>true</turnGravityOff>
   </gazebo>
+  <gazebo reference="thruster_right_dummy">
+    <turnGravityOff>true</turnGravityOff>
+  </gazebo>
   <gazebo reference="thruster_left">
     <turnGravityOff>true</turnGravityOff>

Commit message: Added the left thruster with controllers

File: urdf/asv_base.urdf.xacro (robot description, xacro)
@@ -61,4 +61,16 @@
     <dynamics damping="0.1" friction="0.1" />
   </joint>
+    <link name="thruster_left_dummy">
+    <inertial>
+      <origin rpy="0 0 0" xyz="-4.8522E-05 0.00051157 0.0095278"/>
+      <mass value="0.2183"/>
+      <inertia ixx="9.1096E-05" ixy="3.0619E-09" ixz="-1.6688E-07" iyy="9.0558E-05" iyz="1.2699E-06" izz="1.246E-06"/>
+    </inertial>
+  </link>
+  <joint name="thruster_left_fix" type="fixed">
+    <origin xyz="0 -0.95 1.7088" rpy="1.5708 0 0" />
+    <parent link="base_footprint"/>
+    <child link="thruster_left_dummy"/>
+  </joint>
   <link name="thruster_left">
     <inertial>
@@ -68,5 +80,5 @@
     </inertial>
     <visual>
-      <origin rpy="0 0 0" xyz="0 0 0"/>
+      <origin rpy="0 1.5708 1.5708" xyz="0 0 0"/>
       <geometry>
         <mesh filename="$(arg path)/thruster_left.STL"/>
@@ -85,5 +97,5 @@
   <joint name="body_to_thruster_left" type="continuous">
     <origin rpy="1.5708 0 3.1416" xyz="0.027678 -1.335 0.37124"/>
-    <parent link="base_footprint"/>
+    <parent link="thruster_left_dummy"/>
     <child link="thruster_left"/>
     <axis xyz="0 1 0"/>

Commit message: Added folder worlds for adding future worlds. Also, added the laser sensor to the model of the ASV.

File: urdf/asv_base.urdf.xacro (robot description, xacro)
@@ -52,4 +52,10 @@
       </material>
     </visual>
+    <collision>
+      <origin rpy="0 1.5708 1.5708" xyz="0 0 0"/>
+      <geometry>
+        <mesh filename="$(arg path)/thruster_right.STL"/>
+      </geometry>
+    </collision>
   </link>
   <joint name="body_to_thruster_right" type="continuous">
@@ -496,12 +502,43 @@
     <axis xyz="0 0 0"/>
   </joint>
-  <sensor name="lidar" update_rate="30">
+  <sensor name="lidar" update_rate="50">
     <parent link="lidar" />
     <origin xyz="0 0 0" rpy="0 0 0 " />
     <ray>
-      <horizontal samples="100" resolution="1" min_angle="-1.5708" max_angle="1.5708" />
+      <horizontal samples="100" resolution="1" min_angle="-1.1781" max_angle="1.1781" />
       <vertical samples="1" resolution="1" min_angle="0" max_angle="0"/>
     </ray>
   </sensor>
+  <gazebo reference="lidar">
+    <sensor name="lmssick" type="ray">
+    <pose>0 0 0 0 0 0</pose>
+    <visualize>false</visualize>
+    <update_rate>50</update_rate>
+    <ray>
+      <scan>
+        <horizontal>
+          <samples>100</samples>
+          <resolution>1</resolution>
+          <min_angle>-1.1781</min_angle>
+          <max_angle>1.1781</max_angle>
+        </horizontal>
+      </scan>
+        <range>
+          <min>0.05</min>
+          <max>20</max>
+          <resolution>0.01</resolution>
+        </range>
+        <noise>
+          <type>gaussian</type>
+          <mean>0.0</mean>
+          <stddev>0.01</stddev>
+        </noise>
+    </ray>
+    <plugin name="sicklms" filename="libgazebo_ros_laser.so">
+      <topicName>/asv/laser/scan</topicName>
+      <frameName>lidar</frameName>
+    </plugin>
+  </sensor>
+  </gazebo>
 <transmission name="left_thruster_rotation">
   <type>transmission_interface/SimpleTransmission</type>
