Commit message: Cleaned the package for better readability and understanding

File: urdf/asv_base.xacro (robot description, xacro)
@@ -8,19 +8,22 @@
   </gazebo>
   <xacro:property name="PI" value="3.14159265359" />
-  <xacro:arg name="path" default="package://asv_description/meshes" />
-   <link name="base_footprint">
-    <inertial>
-      <origin rpy="0 0 0" xyz="0.38789 0.59329 1.1865"/>
-      <mass value="2.331"/>
-      <inertia ixx="0" ixy="0" ixz="0" iyy="0" iyz="0" izz="0"/>
-    </inertial>
-    <visual>
-      <origin rpy="0 0 0" xyz="0 0 0"/>
-      <geometry>
-        <mesh filename="$(arg path)/asv.STL"/>
-      </geometry>
+  <xacro:property name="fiber">
       <material name="">
         <color rgba="0.79216 0.81961 0.93333 1"/>
       </material>
+  </xacro:property>
+  <xacro:arg name="path" default="package://asv_description/meshes" />
+   <link name="base_footprint">
+    <inertial>
+      <origin rpy="0 0 0" xyz="0.38789 0.59329 1.1865"/>
+      <mass value="2.331"/>
+      <inertia ixx="0" ixy="0" ixz="0" iyy="0" iyz="0" izz="0"/>
+    </inertial>
+    <visual>
+      <origin rpy="0 0 0" xyz="0 0 0"/>
+      <geometry>
+        <mesh filename="$(arg path)/asv.STL"/>
+      </geometry>
+<xacro:insert_block name="fiber" />
     </visual>
   </link>
@@ -48,7 +51,5 @@
         <mesh filename="$(arg path)/thruster_right.STL"/>
       </geometry>
-      <material name="">
-        <color rgba="0.79216 0.81961 0.93333 1"/>
-      </material>
+<xacro:insert_block name="fiber" />
     </visual>
     <collision>
@@ -90,7 +91,5 @@
         <mesh filename="$(arg path)/thruster_left.STL"/>
       </geometry>
-      <material name="">
-        <color rgba="0.79216 0.81961 0.93333 1"/>
-      </material>
+<xacro:insert_block name="fiber" />
     </visual>
     <collision>
@@ -177,7 +176,5 @@
         <mesh filename="$(arg path)/sensor_pod.STL"/>
       </geometry>
-      <material name="">
-        <color rgba="0.79216 0.81961 0.93333 1"/>
-      </material>
+<xacro:insert_block name="fiber" />
     </visual>
     <collision>
@@ -205,7 +202,5 @@
         <mesh filename="$(arg path)/camera_garmin_mounts.STL"/>
       </geometry>
-      <material name="">
-        <color rgba="0.79216 0.81961 0.93333 1"/>
-      </material>
+<xacro:insert_block name="fiber" />
     </visual>
     <collision>
@@ -233,7 +228,5 @@
         <mesh filename="$(arg path)/garmin.STL"/>
       </geometry>
-      <material name="">
-        <color rgba="0.79216 0.81961 0.93333 1"/>
-      </material>
+<xacro:insert_block name="fiber" />
     </visual>
     <collision>
@@ -289,7 +282,5 @@
         <mesh filename="$(arg path)/lidar.STL"/>
       </geometry>
-      <material name="">
-        <color rgba="0.79216 0.81961 0.93333 1"/>
-      </material>
+<xacro:insert_block name="fiber" />
     </visual>
     <collision>
@@ -317,7 +308,5 @@
         <mesh filename="$(arg path)/kill_switch_2.STL"/>
       </geometry>
-      <material name="">
-        <color rgba="0.79216 0.81961 0.93333 1"/>
-      </material>
+<xacro:insert_block name="fiber" />
     </visual>
     <collision>
@@ -345,7 +334,5 @@
         <mesh filename="$(arg path)/kill_switch_1.STL"/>
       </geometry>
-      <material name="">
-        <color rgba="0.79216 0.81961 0.93333 1"/>
-      </material>
+<xacro:insert_block name="fiber" />
     </visual>
     <collision>
@@ -373,7 +360,5 @@
         <mesh filename="$(arg path)/battery_1.STL"/>
       </geometry>
-      <material name="">
-        <color rgba="0.79216 0.81961 0.93333 1"/>
-      </material>
+<xacro:insert_block name="fiber" />
     </visual>
     <collision>
@@ -401,7 +386,5 @@
         <mesh filename="$(arg path)/battery_2.STL"/>
       </geometry>
-      <material name="">
-        <color rgba="0.79216 0.81961 0.93333 1"/>
-      </material>
+<xacro:insert_block name="fiber" />
     </visual>
     <collision>
@@ -429,7 +412,5 @@
         <mesh filename="$(arg path)/mount.STL"/>
       </geometry>
-      <material name="">
-        <color rgba="0.79216 0.81961 0.93333 1"/>
-      </material>
+<xacro:insert_block name="fiber" />
     </visual>
     <collision>
@@ -457,7 +438,5 @@
         <mesh filename="$(arg path)/rs_232_port.STL"/>
       </geometry>
-      <material name="">
-        <color rgba="0.79216 0.81961 0.93333 1"/>
-      </material>
+<xacro:insert_block name="fiber" />
     </visual>
     <collision>
@@ -485,7 +464,5 @@
         <mesh filename="$(arg path)/status_board.STL"/>
       </geometry>
-      <material name="">
-        <color rgba="0.79216 0.81961 0.93333 1"/>
-      </material>
+<xacro:insert_block name="fiber" />
     </visual>
     <collision>
@@ -512,4 +489,5 @@
   <gazebo reference="lidar">
     <sensor name="lmssick" type="ray">
+      <always_on>1</always_on>
     <pose>0 0 0 0 0 0</pose>
     <visualize>false</visualize>
@@ -559,57 +537,3 @@
   </actuator>
 </transmission>
-  <gazebo reference="base_footprint">
-    <turnGravityOff>true</turnGravityOff>
-  </gazebo>
-  <gazebo reference="thruster_right">
-    <turnGravityOff>true</turnGravityOff>
-  </gazebo>
-  <gazebo reference="thruster_right_dummy">
-    <turnGravityOff>true</turnGravityOff>
-  </gazebo>
-  <gazebo reference="thruster_left">
-    <turnGravityOff>true</turnGravityOff>
-  </gazebo>
-  <gazebo reference="top_body">
-    <turnGravityOff>true</turnGravityOff>
-  </gazebo>
-    <gazebo reference="top_cover">
-    <turnGravityOff>true</turnGravityOff>
-  </gazebo>
-    <gazebo reference="sensor_pod">
-    <turnGravityOff>true</turnGravityOff>
-  </gazebo>
-    <gazebo reference="camera_garmin_mounts">
-    <turnGravityOff>true</turnGravityOff>
-  </gazebo>
-    <gazebo reference="garmin">
-    <turnGravityOff>true</turnGravityOff>
-  </gazebo>
-    <gazebo reference="camera">
-    <turnGravityOff>true</turnGravityOff>
-  </gazebo>
-    <gazebo reference="lidar">
-    <turnGravityOff>true</turnGravityOff>
-  </gazebo>
-    <gazebo reference="kill_switch_1">
-    <turnGravityOff>true</turnGravityOff>
-  </gazebo>
-    <gazebo reference="kill_switch_2">
-    <turnGravityOff>true</turnGravityOff>
-  </gazebo>
-    <gazebo reference="battery_1">
-    <turnGravityOff>true</turnGravityOff>
-  </gazebo>
-    <gazebo reference="battery_2">
-    <turnGravityOff>true</turnGravityOff>
-  </gazebo>
-    <gazebo reference="mount">
-    <turnGravityOff>true</turnGravityOff>
-  </gazebo>
-    <gazebo reference="rs_232_port">
-    <turnGravityOff>true</turnGravityOff>
-  </gazebo>
-    <gazebo reference="status_board">
-    <turnGravityOff>true</turnGravityOff>
-  </gazebo>
 </robot>

Commit message: Cleaned the package.xml file and gazebo.launch file for brevity

File: urdf/asv_base.xacro (robot description, xacro)
@@ -479,39 +479,13 @@
     <axis xyz="0 0 0"/>
   </joint>
-  <sensor name="lidar" update_rate="50">
+  <sensor name="lidar" update_rate="50" type="laser">
     <parent link="lidar" />
-    <origin xyz="0 0 0" rpy="0 0 0 " />
-    <ray>
-      <horizontal samples="100" resolution="1" min_angle="-1.1781" max_angle="1.1781" />
-      <vertical samples="1" resolution="1" min_angle="0" max_angle="0"/>
-    </ray>
+    <origin xyz="0 0 0" rpy="0 0 0" />
+    <ray />
   </sensor>
-  <gazebo reference="lidar">
-    <sensor name="lmssick" type="ray">
-      <always_on>1</always_on>
-    <pose>0 0 0 0 0 0</pose>
-    <visualize>false</visualize>
+<gazebo reference="lidar">
+  <sensor name="lmssick" type="ray">
     <update_rate>50</update_rate>
-    <ray>
-      <scan>
-        <horizontal>
-          <samples>100</samples>
-          <resolution>1</resolution>
-          <min_angle>-1.1781</min_angle>
-          <max_angle>1.1781</max_angle>
-        </horizontal>
-      </scan>
-        <range>
-          <min>0.05</min>
-          <max>20</max>
-          <resolution>0.01</resolution>
-        </range>
-        <noise>
-          <type>gaussian</type>
-          <mean>0.0</mean>
-          <stddev>0.01</stddev>
-        </noise>
-    </ray>
-    <plugin name="sicklms" filename="libgazebo_ros_laser.so">
+    <plugin name="lidar" filename="libgazebo_ros_laser.so">
       <topicName>/asv/laser/scan</topicName>
       <frameName>lidar</frameName>

Commit message: Added controllers and sensors xacro for modularity

File: urdf/asv_base.xacro (robot description, xacro)
@@ -1,20 +1,29 @@
 <?xml version="1.0"?>
 <robot xmlns:xacro="http://www.ros.org/wiki/xacro" name="asv_description">
-  <gazebo>
-    <plugin name="ros_control" filename="libgazebo_ros_control.so">
-      <robotNamespace>/asv</robotNamespace>
-      <robotSimType>gazebo_ros_control/DefaultRobotHWSim</robotSimType>
-    </plugin>
+  <xacro:arg name="path" default="package://asv_description/meshes" />
+    <link name="base_footprint">
+    <inertial>
+      <mass value="0.0001"/>
+      <origin xyz="0 0 0"/>
+      <inertia ixx="0.0001" ixy="0.0" ixz="0.0" iyy="0.0001" iyz="0.0" izz="0.0001"/>
+    </inertial>
+    <visual>
+      <origin rpy="0 0 0" xyz="0 0 0"/>
+      <geometry>
+        <box size="0.001 0.001 0.001"/>
+      </geometry>
+    </visual>
+  </link>
+  <gazebo reference="base_footprint">
+    <turnGravityOff>false</turnGravityOff>
   </gazebo>
-  <xacro:property name="PI" value="3.14159265359" />
-  <xacro:property name="fiber">
-      <material name="">
-        <color rgba="0.79216 0.81961 0.93333 1"/>
-      </material>
-  </xacro:property>
-  <xacro:arg name="path" default="package://asv_description/meshes" />
-   <link name="base_footprint">
-    <inertial>
-      <origin rpy="0 0 0" xyz="0.38789 0.59329 1.1865"/>
+  <joint name="base_footprint_joint" type="fixed">
+    <origin rpy="0 0 0" xyz="0 0 0"/>
+    <parent link="base_footprint"/>
+    <child link="base_link"/>
+  </joint>
+   <link name="base_link">
+    <inertial>
+      <origin rpy="0 0 0" xyz="0 0 0"/>
       <mass value="2.331"/>
       <inertia ixx="0" ixy="0" ixz="0" iyy="0" iyz="0" izz="0"/>
@@ -37,5 +46,5 @@
   <joint name="thruster_right_fix" type="fixed">
     <origin xyz="0 -0.95 1.7088" rpy="1.5708 0 0" />
-    <parent link="base_footprint"/>
+    <parent link="base_link"/>
     <child link="thruster_right_dummy"/>
   </joint>
@@ -54,7 +63,7 @@
     </visual>
     <collision>
-      <origin rpy="0 1.5708 1.5708" xyz="0 0 0"/>
-      <geometry>
-        <mesh filename="$(arg path)/thruster_right.STL"/>
+      <origin rpy="0 0 0" xyz="0 0 0"/>
+      <geometry>
+        <cylinder radius="0.05" length="0.15" />
       </geometry>
     </collision>
@@ -77,5 +86,5 @@
   <joint name="thruster_left_fix" type="fixed">
     <origin xyz="0 -0.95 1.7088" rpy="1.5708 0 0" />
-    <parent link="base_footprint"/>
+    <parent link="base_link"/>
     <child link="thruster_left_dummy"/>
   </joint>
@@ -123,14 +132,8 @@
       </material>
     </visual>
-    <collision>
-      <origin rpy="0 0 0" xyz="0 0 0"/>
-      <geometry>
-        <mesh filename="$(arg path)/top_body.STL"/>
-      </geometry>
-    </collision>
   </link>
   <joint name="asv_to_top_body" type="fixed">
     <origin rpy="1.5708 0 0" xyz="0.38708 -1.0625 0.60681"/>
-    <parent link="base_footprint"/>
+    <parent link="base_link"/>
     <child link="top_body"/>
     <axis xyz="0 0 0"/>
@@ -151,10 +154,4 @@
       </material>
     </visual>
-    <collision>
-      <origin xyz="0 0 0" rpy="0 0 0" />
-      <geometry>
-        <mesh filename="$(arg path)/top_cover.STL" />
-      </geometry>
-    </collision>
   </link>
   <joint name="top_body_to_cover" type="fixed">
@@ -178,10 +175,4 @@
 <xacro:insert_block name="fiber" />
     </visual>
-    <collision>
-      <origin rpy="0 0 0" xyz="0 0 0"/>
-      <geometry>
-        <mesh filename="$(arg path)/sensor_pod.STL"/>
-      </geometry>
-    </collision>
   </link>
   <joint name="top_to_sensor_pod" type="fixed">
@@ -204,10 +195,4 @@
 <xacro:insert_block name="fiber" />
     </visual>
-    <collision>
-      <origin rpy="0 0 0" xyz="0 0 0"/>
-      <geometry>
-        <mesh filename="$(arg path)/camera_garmin_mounts.STL"/>
-      </geometry>
-    </collision>
   </link>
   <joint name="pod_to_mounts" type="fixed">
@@ -230,10 +215,4 @@
 <xacro:insert_block name="fiber" />
     </visual>
-    <collision>
-      <origin rpy="3.141592653589793 0 0" xyz="0 0 0"/>
-      <geometry>
-        <mesh filename="$(arg path)/garmin.STL"/>
-      </geometry>
-    </collision>
   </link>
   <joint name="mount_to_garmin" type="fixed">
@@ -258,10 +237,4 @@
       </material>
     </visual>
-    <collision>
-      <origin rpy="0 0 0" xyz="0 0 0"/>
-      <geometry>
-        <mesh filename="$(arg path)/camera.STL"/>
-      </geometry>
-    </collision>
   </link>
   <joint name="mount_to_camera" type="fixed">
@@ -284,10 +257,4 @@
 <xacro:insert_block name="fiber" />
     </visual>
-    <collision>
-      <origin rpy="0 0 0" xyz="0 0 0"/>
-      <geometry>
-        <mesh filename="$(arg path)/lidar.STL"/>
-      </geometry>
-    </collision>
   </link>
   <joint name="pod_to_lidar" type="fixed">
@@ -310,10 +277,4 @@
 <xacro:insert_block name="fiber" />
     </visual>
-    <collision>
-      <origin rpy="0 0 0" xyz="0 0 0"/>
-      <geometry>
-        <mesh filename="$(arg path)/kill_switch_2.STL"/>
-      </geometry>
-    </collision>
   </link>
   <joint name="top_to_kill_2" type="fixed">
@@ -336,10 +297,4 @@
 <xacro:insert_block name="fiber" />
     </visual>
-    <collision>
-      <origin rpy="0 0 0" xyz="0 0 0"/>
-      <geometry>
-        <mesh filename="$(arg path)/kill_switch_1.STL"/>
-      </geometry>
-    </collision>
   </link>
   <joint name="top_to_kill_1" type="fixed">
@@ -362,14 +317,8 @@
 <xacro:insert_block name="fiber" />
     </visual>
-    <collision>
-      <origin rpy="0 0 0" xyz="0 0 0"/>
-      <geometry>
-        <mesh filename="$(arg path)/battery_1.STL"/>
-      </geometry>
-    </collision>
   </link>
   <joint name="body_to_battery" type="fixed">
     <origin rpy="3.1416 0 0" xyz="0.38768 -1.5211 0.59834"/>
-    <parent link="base_footprint"/>
+    <parent link="base_link"/>
     <child link="battery_1"/>
     <axis xyz="0 0 0"/>
@@ -388,10 +337,4 @@
 <xacro:insert_block name="fiber" />
     </visual>
-    <collision>
-      <origin rpy="0 0 0" xyz="0 0 0"/>
-      <geometry>
-        <mesh filename="$(arg path)/battery_2.STL"/>
-      </geometry>
-    </collision>
   </link>
   <joint name="battery_1_to_battery_2" type="fixed">
@@ -414,14 +357,8 @@
 <xacro:insert_block name="fiber" />
     </visual>
-    <collision>
-      <origin rpy="0 0 0" xyz="0 0 0"/>
-      <geometry>
-        <mesh filename="$(arg path)/mount.STL"/>
-      </geometry>
-    </collision>
   </link>
   <joint name="body_to_mount" type="fixed">
     <origin rpy="1.5708 0 0" xyz="0.38768 -1.2531 0.56334"/>
-    <parent link="base_footprint"/>
+    <parent link="base_link"/>
     <child link="mount"/>
     <axis xyz="0 0 0"/>
@@ -440,10 +377,4 @@
 <xacro:insert_block name="fiber" />
     </visual>
-    <collision>
-      <origin rpy="0 0 0" xyz="0 0 0"/>
-      <geometry>
-        <mesh filename="$(arg path)/rs_232_port.STL"/>
-      </geometry>
-    </collision>
   </link>
   <joint name="mount_to_port" type="fixed">
@@ -466,10 +397,4 @@
 <xacro:insert_block name="fiber" />
     </visual>
-    <collision>
-      <origin rpy="0 0 0" xyz="0 0 0"/>
-      <geometry>
-        <mesh filename="$(arg path)/status_board.STL"/>
-      </geometry>
-    </collision>
   </link>
   <joint name="mount_to_status_board" type="fixed">
@@ -479,35 +404,5 @@
     <axis xyz="0 0 0"/>
   </joint>
-  <sensor name="lidar" update_rate="50" type="laser">
-    <parent link="lidar" />
-    <origin xyz="0 0 0" rpy="0 0 0" />
-    <ray />
-  </sensor>
-<gazebo reference="lidar">
-  <sensor name="lmssick" type="ray">
-    <update_rate>50</update_rate>
-    <plugin name="lidar" filename="libgazebo_ros_laser.so">
-      <topicName>/asv/laser/scan</topicName>
-      <frameName>lidar</frameName>
-    </plugin>
-  </sensor>
-  </gazebo>
-<transmission name="left_thruster_rotation">
-  <type>transmission_interface/SimpleTransmission</type>
-  <joint name="body_to_thruster_left">
-    <hardwareInterface>hardware_interface/EffortJointInterface</hardwareInterface>
-  </joint>
-  <actuator name="left_thruster_actuator">
-    <mechanicalReduction>1</mechanicalReduction>
-  </actuator>
-</transmission>
-<transmission name="right_thruster_rotation">
-  <type>transmission_interface/SimpleTransmission</type>
-  <joint name="body_to_thruster_right">
-    <hardwareInterface>hardware_interface/EffortJointInterface</hardwareInterface>
-  </joint>
-  <actuator name="right_thruster_actuator">
-    <mechanicalReduction>1</mechanicalReduction>
-  </actuator>
-</transmission>
+<xacro:include filename="$(find asv_description)/urdf/asv_sensors.xacro" />
+<xacro:include filename="$(find asv_description)/urdf/asv_controllers.xacro" />
 </robot>
