Commit message: Added properties and sim xacro files for turtlebot package similarity

File: urdf/asv_base.xacro (robot description, xacro)
@@ -1,6 +1,8 @@
 <?xml version="1.0"?>
-<robot xmlns:xacro="http://www.ros.org/wiki/xacro" name="asv_description">
-  <xacro:arg name="path" default="package://asv_description/meshes" />
-    <link name="base_footprint">
+<robot name="asv_description" xmlns:xacro="http://www.ros.org/wiki/xacro">
+ <xacro:arg default="package://asv_description/meshes" name="path"/>
+  <xacro:include filename="$(find asv_description)/urdf/common_properties.xacro"/>
+  <xacro:include filename="$(find asv_description)/urdf/sim.xacro"/>
+  <link name="base_footprint">
     <inertial>
       <mass value="0.0001"/>
@@ -15,7 +17,4 @@
     </visual>
   </link>
-  <gazebo reference="base_footprint">
-    <turnGravityOff>false</turnGravityOff>
-  </gazebo>
   <joint name="base_footprint_joint" type="fixed">
     <origin rpy="0 0 0" xyz="0 0 0"/>
@@ -23,5 +22,5 @@
     <child link="base_link"/>
   </joint>
-   <link name="base_link">
+  <link name="base_link">
     <inertial>
       <origin rpy="0 0 0" xyz="0 0 0"/>
@@ -34,5 +33,5 @@
         <mesh filename="$(arg path)/asv.STL"/>
       </geometry>
-<xacro:insert_block name="fiber" />
+      <xacro:insert_block name="fiber"/>
     </visual>
   </link>
@@ -45,5 +44,5 @@
   </link>
   <joint name="thruster_right_fix" type="fixed">
-    <origin xyz="0 -0.95 1.7088" rpy="1.5708 0 0" />
+    <origin rpy="1.5708 0 0" xyz="0 -0.95 1.7088"/>
     <parent link="base_link"/>
     <child link="thruster_right_dummy"/>
@@ -60,10 +59,10 @@
         <mesh filename="$(arg path)/thruster_right.STL"/>
       </geometry>
-<xacro:insert_block name="fiber" />
+      <xacro:insert_block name="fiber"/>
     </visual>
     <collision>
       <origin rpy="0 0 0" xyz="0 0 0"/>
       <geometry>
-        <cylinder radius="0.05" length="0.15" />
+        <cylinder length="0.15" radius="0.05"/>
       </geometry>
     </collision>
@@ -74,8 +73,8 @@
     <child link="thruster_right"/>
     <axis xyz="0 -1 0"/>
-       <limit effort="30" velocity="1.0" lower="-32000" upper="32000" />
-    <dynamics damping="0.1" friction="0.1" />
-  </joint>
-    <link name="thruster_left_dummy">
+    <limit effort="30" lower="-32000" upper="32000" velocity="1.0"/>
+    <dynamics damping="0.1" friction="0.1"/>
+  </joint>
+  <link name="thruster_left_dummy">
     <inertial>
       <origin rpy="0 0 0" xyz="-4.8522E-05 0.00051157 0.0095278"/>
@@ -85,5 +84,5 @@
   </link>
   <joint name="thruster_left_fix" type="fixed">
-    <origin xyz="0 -0.95 1.7088" rpy="1.5708 0 0" />
+    <origin rpy="1.5708 0 0" xyz="0 -0.95 1.7088"/>
     <parent link="base_link"/>
     <child link="thruster_left_dummy"/>
@@ -100,5 +99,5 @@
         <mesh filename="$(arg path)/thruster_left.STL"/>
       </geometry>
-<xacro:insert_block name="fiber" />
+      <xacro:insert_block name="fiber"/>
     </visual>
     <collision>
@@ -114,6 +113,6 @@
     <child link="thruster_left"/>
     <axis xyz="0 1 0"/>
-       <limit effort="30" velocity="1.0" lower="-32000" upper="32000" />
-    <dynamics damping="0.1" friction="0.1" />
+    <limit effort="30" lower="-32000" upper="32000" velocity="1.0"/>
+    <dynamics damping="0.1" friction="0.1"/>
   </joint>
   <link name="top_body">
@@ -141,24 +140,24 @@
   <link name="top_cover">
     <inertial>
-      <origin xyz="2.7931E-06 -0.018976 0.0015" rpy="0 0 0" />
-      <mass value="0.43537" />
-      <inertia ixx="0" ixy="0" ixz="0" iyy="0" iyz="0" izz="0" />
-    </inertial>
-    <visual>
-      <origin xyz="0 0 0" rpy="0 0 0" />
-      <geometry>
-        <mesh filename="$(arg path)/top_cover.STL" />
+      <origin rpy="0 0 0" xyz="2.7931E-06 -0.018976 0.0015"/>
+      <mass value="0.43537"/>
+      <inertia ixx="0" ixy="0" ixz="0" iyy="0" iyz="0" izz="0"/>
+    </inertial>
+    <visual>
+      <origin rpy="0 0 0" xyz="0 0 0"/>
+      <geometry>
+        <mesh filename="$(arg path)/top_cover.STL"/>
       </geometry>
       <material name="">
-        <color rgba="0.79216 0.81961 0.93333 1" />
+        <color rgba="0.79216 0.81961 0.93333 1"/>
       </material>
     </visual>
   </link>
   <joint name="top_body_to_cover" type="fixed">
-    <origin xyz="0.00059952 0.19104 0.1763" rpy="-1.5708 0 0" />
-    <parent link="top_body" />
-    <child link="top_cover" />
-    <axis xyz="0 0 1" />
-    <limit lower="0" upper="0.2" effort="0" velocity="0" />
+    <origin rpy="-1.5708 0 0" xyz="0.00059952 0.19104 0.1763"/>
+    <parent link="top_body"/>
+    <child link="top_cover"/>
+    <axis xyz="0 0 1"/>
+    <limit effort="0" lower="0" upper="0.2" velocity="0"/>
   </joint>
   <link name="sensor_pod">
@@ -173,5 +172,5 @@
         <mesh filename="$(arg path)/sensor_pod.STL"/>
       </geometry>
-<xacro:insert_block name="fiber" />
+      <xacro:insert_block name="fiber"/>
     </visual>
   </link>
@@ -193,5 +192,5 @@
         <mesh filename="$(arg path)/camera_garmin_mounts.STL"/>
       </geometry>
-<xacro:insert_block name="fiber" />
+      <xacro:insert_block name="fiber"/>
     </visual>
   </link>
@@ -213,5 +212,5 @@
         <mesh filename="$(arg path)/garmin.STL"/>
       </geometry>
-<xacro:insert_block name="fiber" />
+      <xacro:insert_block name="fiber"/>
     </visual>
   </link>
@@ -255,5 +254,5 @@
         <mesh filename="$(arg path)/lidar.STL"/>
       </geometry>
-<xacro:insert_block name="fiber" />
+      <xacro:insert_block name="fiber"/>
     </visual>
   </link>
@@ -275,5 +274,5 @@
         <mesh filename="$(arg path)/kill_switch_2.STL"/>
       </geometry>
-<xacro:insert_block name="fiber" />
+      <xacro:insert_block name="fiber"/>
     </visual>
   </link>
@@ -295,5 +294,5 @@
         <mesh filename="$(arg path)/kill_switch_1.STL"/>
       </geometry>
-<xacro:insert_block name="fiber" />
+      <xacro:insert_block name="fiber"/>
     </visual>
   </link>
@@ -315,5 +314,5 @@
         <mesh filename="$(arg path)/battery_1.STL"/>
       </geometry>
-<xacro:insert_block name="fiber" />
+      <xacro:insert_block name="fiber"/>
     </visual>
   </link>
@@ -335,5 +334,5 @@
         <mesh filename="$(arg path)/battery_2.STL"/>
       </geometry>
-<xacro:insert_block name="fiber" />
+      <xacro:insert_block name="fiber"/>
     </visual>
   </link>
@@ -355,5 +354,5 @@
         <mesh filename="$(arg path)/mount.STL"/>
       </geometry>
-<xacro:insert_block name="fiber" />
+      <xacro:insert_block name="fiber"/>
     </visual>
   </link>
@@ -375,5 +374,5 @@
         <mesh filename="$(arg path)/rs_232_port.STL"/>
       </geometry>
-<xacro:insert_block name="fiber" />
+      <xacro:insert_block name="fiber"/>
     </visual>
   </link>
@@ -395,5 +394,5 @@
         <mesh filename="$(arg path)/status_board.STL"/>
       </geometry>
-<xacro:insert_block name="fiber" />
+      <xacro:insert_block name="fiber"/>
     </visual>
   </link>
@@ -404,5 +403,5 @@
     <axis xyz="0 0 0"/>
   </joint>
-<xacro:include filename="$(find asv_description)/urdf/asv_sensors.xacro" />
-<xacro:include filename="$(find asv_description)/urdf/asv_controllers.xacro" />
+  <xacro:include filename="$(find asv_description)/urdf/asv_sensors.xacro"/>
+  <xacro:include filename="$(find asv_description)/urdf/asv_controllers.xacro"/>
 </robot>

File: urdf/asv_controllers.xacro (robot description, xacro)
@@ -1,3 +1,3 @@
-  <?xml version="1.0"?>
+<?xml version="1.0"?>
 <robot xmlns:xacro="http://www.ros.org/wiki/xacro" name="controllers">
 <transmission name="left_thruster_rotation">

Commit message: Added new model imported from SolidWorks with fixed origin.

File: urdf/asv_base.xacro (robot description, xacro)
@@ -1,402 +1,294 @@
 <?xml version="1.0"?>
 <robot name="asv_description" xmlns:xacro="http://www.ros.org/wiki/xacro">
-  <link name="base_footprint">
-    <inertial>
-      <mass value="0.0001"/>
-      <origin xyz="0 0 0"/>
-      <inertia ixx="0.0001" ixy="0.0" ixz="0.0" iyy="0.0001" iyz="0.0" izz="0.0001"/>
-    </inertial>
-    <visual>
-      <origin rpy="0 0 0" xyz="0 0 0"/>
-      <geometry>
-        <box size="0.001 0.001 0.001"/>
-      </geometry>
-    </visual>
-  </link>
-  <joint name="base_footprint_joint" type="fixed">
-    <origin rpy="0 0 0" xyz="0 0 0"/>
-    <parent link="base_footprint"/>
-    <child link="base_link"/>
-  </joint>
-  <link name="base_link">
-    <inertial>
-      <origin rpy="0 0 0" xyz="0 0 0"/>
-      <mass value="2.331"/>
-      <inertia ixx="0" ixy="0" ixz="0" iyy="0" iyz="0" izz="0"/>
-    </inertial>
-    <visual>
-      <origin rpy="0 0 0" xyz="0 0 0"/>
-      <geometry>
-        <mesh filename="$(arg path)/asv.STL"/>
-      </geometry>
-      <xacro:insert_block name="fiber"/>
-    </visual>
-  </link>
-  <link name="thruster_right_dummy">
-    <inertial>
-      <origin rpy="0 0 0" xyz="-4.8522E-05 0.00051157 0.0095278"/>
-      <mass value="0.2183"/>
-      <inertia ixx="9.1096E-05" ixy="3.0619E-09" ixz="-1.6688E-07" iyy="9.0558E-05" iyz="1.2699E-06" izz="1.246E-06"/>
-    </inertial>
-  </link>
-  <joint name="thruster_right_fix" type="fixed">
-    <origin rpy="1.5708 0 0" xyz="0 -0.95 1.7088"/>
-    <parent link="base_link"/>
-    <child link="thruster_right_dummy"/>
-  </joint>
-  <link name="thruster_right">
-    <inertial>
-      <origin rpy="0 0 0" xyz="-4.8522E-05 0.00051157 0.0095278"/>
-      <mass value="0.2183"/>
-      <inertia ixx="9.1096E-05" ixy="3.0619E-09" ixz="-1.6688E-07" iyy="9.0558E-05" iyz="1.2699E-06" izz="1.246E-06"/>
-    </inertial>
-    <visual>
-      <origin rpy="0 1.5708 1.5708" xyz="0 0 0"/>
-      <geometry>
-        <mesh filename="$(arg path)/thruster_right.STL"/>
-      </geometry>
-      <xacro:insert_block name="fiber"/>
-    </visual>
-    <collision>
-      <origin rpy="0 0 0" xyz="0 0 0"/>
-      <geometry>
-        <cylinder length="0.15" radius="0.05"/>
-      </geometry>
-    </collision>
-  </link>
-  <joint name="body_to_thruster_right" type="continuous">
-    <origin rpy="1.5708 0 3.1416" xyz="0.74762 -1.335 0.37124"/>
-    <parent link="thruster_right_dummy"/>
-    <child link="thruster_right"/>
-    <axis xyz="0 -1 0"/>
-    <limit effort="30" lower="-32000" upper="32000" velocity="1.0"/>
-    <dynamics damping="0.1" friction="0.1"/>
-  </joint>
-  <link name="thruster_left_dummy">
-    <inertial>
-      <origin rpy="0 0 0" xyz="-4.8522E-05 0.00051157 0.0095278"/>
-      <mass value="0.2183"/>
-      <inertia ixx="9.1096E-05" ixy="3.0619E-09" ixz="-1.6688E-07" iyy="9.0558E-05" iyz="1.2699E-06" izz="1.246E-06"/>
-    </inertial>
-  </link>
-  <joint name="thruster_left_fix" type="fixed">
-    <origin rpy="1.5708 0 0" xyz="0 -0.95 1.7088"/>
-    <parent link="base_link"/>
-    <child link="thruster_left_dummy"/>
-  </joint>
-  <link name="thruster_left">
-    <inertial>
-      <origin rpy="0 0 0" xyz="-4.8521E-05 0.00051157 0.0095278"/>
-      <mass value="0.2183"/>
-      <inertia ixx="9.1096E-05" ixy="3.0619E-09" ixz="-1.6688E-07" iyy="9.0558E-05" iyz="1.2699E-06" izz="1.246E-06"/>
-    </inertial>
-    <visual>
-      <origin rpy="0 1.5708 1.5708" xyz="0 0 0"/>
-      <geometry>
-        <mesh filename="$(arg path)/thruster_left.STL"/>
-      </geometry>
-      <xacro:insert_block name="fiber"/>
-    </visual>
-    <collision>
-      <origin rpy="0 0 0" xyz="0 0 0"/>
-      <geometry>
-        <mesh filename="$(arg path)/thruster_left.STL"/>
-      </geometry>
-    </collision>
-  </link>
-  <joint name="body_to_thruster_left" type="continuous">
-    <origin rpy="1.5708 0 3.1416" xyz="0.027678 -1.335 0.37124"/>
-    <parent link="thruster_left_dummy"/>
-    <child link="thruster_left"/>
-    <axis xyz="0 1 0"/>
-    <limit effort="30" lower="-32000" upper="32000" velocity="1.0"/>
-    <dynamics damping="0.1" friction="0.1"/>
-  </joint>
-  <link name="top_body">
-    <inertial>
-      <origin rpy="0 0 0" xyz="-3.2569E-05 0.15165 0.037912"/>
-      <mass value="1.6252"/>
-      <inertia ixx="0" ixy="0" ixz="0" iyy="0" iyz="0" izz="0"/>
-    </inertial>
-    <visual>
-      <origin rpy="0 0 0" xyz="0 0 0"/>
-      <geometry>
-        <mesh filename="$(arg path)/top_body.STL"/>
-      </geometry>
-      <material name="">
-        <color rgba="1 1 0.50196 1"/>
-      </material>
-    </visual>
-  </link>
-  <joint name="asv_to_top_body" type="fixed">
-    <origin rpy="1.5708 0 0" xyz="0.38708 -1.0625 0.60681"/>
-    <parent link="base_link"/>
-    <child link="top_body"/>
-    <axis xyz="0 0 0"/>
-  </joint>
-  <link name="top_cover">
-    <inertial>
-      <origin rpy="0 0 0" xyz="2.7931E-06 -0.018976 0.0015"/>
-      <mass value="0.43537"/>
-      <inertia ixx="0" ixy="0" ixz="0" iyy="0" iyz="0" izz="0"/>
-    </inertial>
-    <visual>
-      <origin rpy="0 0 0" xyz="0 0 0"/>
-      <geometry>
-        <mesh filename="$(arg path)/top_cover.STL"/>
-      </geometry>
-      <material name="">
-        <color rgba="0.79216 0.81961 0.93333 1"/>
-      </material>
-    </visual>
-  </link>
-  <joint name="top_body_to_cover" type="fixed">
-    <origin rpy="-1.5708 0 0" xyz="0.00059952 0.19104 0.1763"/>
-    <parent link="top_body"/>
-    <child link="top_cover"/>
-    <axis xyz="0 0 1"/>
-    <limit effort="0" lower="0" upper="0.2" velocity="0"/>
-  </joint>
-  <link name="sensor_pod">
-    <inertial>
-      <origin rpy="0 0 0" xyz="-0.029193 -0.040604 -0.010551"/>
-      <mass value="0.06495"/>
-      <inertia ixx="0.0016814" ixy="-1.4742E-07" ixz="-3.6677E-05" iyy="0.0016822" iyz="-6.7581E-06" izz="8.2722E-07"/>
-    </inertial>
-    <visual>
-      <origin rpy="0 0 0" xyz="0 0 0"/>
-      <geometry>
-        <mesh filename="$(arg path)/sensor_pod.STL"/>
-      </geometry>
-      <xacro:insert_block name="fiber"/>
-    </visual>
-  </link>
-  <joint name="top_to_sensor_pod" type="fixed">
-    <origin rpy="0 1.5708 0" xyz="0 0.2547 -0.47015"/>
-    <parent link="top_body"/>
-    <child link="sensor_pod"/>
-    <axis xyz="0 0 1"/>
-  </joint>
-  <link name="camera_garmin_mounts">
-    <inertial>
-      <origin rpy="0 0 0" xyz="0.0027436 0.024777 0.009305"/>
-      <mass value="0.011757"/>
-      <inertia ixx="0.0001482" ixy="1.0861E-19" ixz="-3.2822E-19" iyy="0.00013357" iyz="4.4199E-05" izz="1.4626E-05"/>
-    </inertial>
-    <visual>
-      <origin rpy="0 0 0" xyz="0 0 0"/>
-      <geometry>
-        <mesh filename="$(arg path)/camera_garmin_mounts.STL"/>
-      </geometry>
-      <xacro:insert_block name="fiber"/>
-    </visual>
-  </link>
-  <joint name="pod_to_mounts" type="fixed">
-    <origin rpy="0 -1.5708 0" xyz="-0.039919 0.069841 0"/>
-    <parent link="sensor_pod"/>
-    <child link="camera_garmin_mounts"/>
-    <axis xyz="1 0 0"/>
-  </joint>
-  <link name="garmin">
-    <inertial>
-      <origin rpy="3.141592653589793 0 0" xyz="0 0.023342 0"/>
-      <mass value="0.03356"/>
-      <inertia ixx="0" ixy="0" ixz="0" iyy="0" iyz="0" izz="0"/>
-    </inertial>
-    <visual>
-      <origin rpy="3.141592653589793 0 0" xyz="0 0 0"/>
-      <geometry>
-        <mesh filename="$(arg path)/garmin.STL"/>
-      </geometry>
-      <xacro:insert_block name="fiber"/>
-    </visual>
-  </link>
-  <joint name="mount_to_garmin" type="fixed">
-    <origin rpy="3.141592653589793 -0.18516 0" xyz="0.0027436 0.026 0.059"/>
-    <parent link="camera_garmin_mounts"/>
-    <child link="garmin"/>
-    <axis xyz="0 0 0"/>
-  </joint>
-  <link name="camera">
-    <inertial>
-      <origin rpy="0 0 0" xyz="-2.8934E-05 -0.010178 0.021487"/>
-      <mass value="0.0041091"/>
-      <inertia ixx="1.4847E-05" ixy="-3.2519E-08" ixz="-1.1631E-08" iyy="3.365E-06" iyz="-4.1204E-06" izz="1.1483E-05"/>
-    </inertial>
-    <visual>
-      <origin rpy="0 0 0" xyz="0 0 0"/>
-      <geometry>
-        <mesh filename="$(arg path)/camera.STL"/>
-      </geometry>
-      <material name="">
-        <color rgba="0.019608 0.019608 0.019608 1"/>
-      </material>
-    </visual>
-  </link>
-  <joint name="mount_to_camera" type="fixed">
-    <origin rpy="3.1167 0.020214 3.1416" xyz="0.002382 0.14006 -0.050118"/>
-    <parent link="camera_garmin_mounts"/>
-    <child link="camera"/>
-    <axis xyz="0 0 0"/>
-  </joint>
-  <link name="lidar">
-    <inertial>
-      <origin rpy="0 0 0" xyz="0.00017493 -0.020457 0.00018726"/>
-      <mass value="8.4876E-05"/>
-      <inertia ixx="7.4827E-08" ixy="1.3927E-09" ixz="-5.2849E-10" iyy="1.4091E-07" iyz="1.6125E-09" izz="7.4592E-08"/>
-    </inertial>
-    <visual>
-      <origin rpy="0 0 0" xyz="0 0 0"/>
-      <geometry>
-        <mesh filename="$(arg path)/lidar.STL"/>
-      </geometry>
-      <xacro:insert_block name="fiber"/>
-    </visual>
-  </link>
-  <joint name="pod_to_lidar" type="fixed">
-    <origin rpy="2.9322 -1.5708 0" xyz="0.12046 0.10702 0.0022421"/>
-    <parent link="sensor_pod"/>
-    <child link="lidar"/>
-    <axis xyz="0 0 0"/>
-  </joint>
-  <link name="kill_switch_2">
-    <inertial>
-      <origin rpy="0 0 0" xyz="0.21906 0.04363 0.013308"/>
-      <mass value="0.0048397"/>
-      <inertia ixx="0" ixy="0" ixz="0" iyy="0" iyz="0" izz="0"/>
-    </inertial>
-    <visual>
-      <origin rpy="0 0 0" xyz="0 0 0"/>
-      <geometry>
-        <mesh filename="$(arg path)/kill_switch_2.STL"/>
-      </geometry>
-      <xacro:insert_block name="fiber"/>
-    </visual>
-  </link>
-  <joint name="top_to_kill_2" type="fixed">
-    <origin rpy="1.5708 0.5236 -1.5708" xyz="0.34081 0.37001 0.43324"/>
-    <parent link="top_body"/>
-    <child link="kill_switch_2"/>
-    <axis xyz="0 0 0"/>
-  </joint>
-  <link name="kill_switch_1">
-    <inertial>
-      <origin rpy="0 0 0" xyz="0.21906 0.04363 0.013308"/>
-      <mass value="0.0048397"/>
-      <inertia ixx="0" ixy="0" ixz="0" iyy="0" iyz="0" izz="0"/>
-    </inertial>
-    <visual>
-      <origin rpy="0 0 0" xyz="0 0 0"/>
-      <geometry>
-        <mesh filename="$(arg path)/kill_switch_1.STL"/>
-      </geometry>
-      <xacro:insert_block name="fiber"/>
-    </visual>
-  </link>
-  <joint name="top_to_kill_1" type="fixed">
-    <origin rpy="-1.5708 0.5236 -1.5708" xyz="-0.34081 0.32638 0.50881"/>
-    <parent link="top_body"/>
-    <child link="kill_switch_1"/>
-    <axis xyz="0 0 0"/>
-  </joint>
-  <link name="battery_1">
-    <inertial>
-      <origin rpy="0 0 0" xyz="-5.5511E-17 0.0185 0"/>
-      <mass value="0.4921"/>
-      <inertia ixx="0" ixy="0" ixz="0" iyy="0" iyz="0" izz="0"/>
-    </inertial>
-    <visual>
-      <origin rpy="0 0 0" xyz="0 0 0"/>
-      <geometry>
-        <mesh filename="$(arg path)/battery_1.STL"/>
-      </geometry>
-      <xacro:insert_block name="fiber"/>
-    </visual>
-  </link>
-  <joint name="body_to_battery" type="fixed">
-    <origin rpy="3.1416 0 0" xyz="0.38768 -1.5211 0.59834"/>
-    <parent link="base_link"/>
-    <child link="battery_1"/>
-    <axis xyz="0 0 0"/>
-  </joint>
-  <link name="battery_2">
-    <inertial>
-      <origin rpy="0 0 0" xyz="-5.5511E-17 0.0185 0"/>
-      <mass value="0.4921"/>
-      <inertia ixx="0" ixy="0" ixz="0" iyy="0" iyz="0" izz="0"/>
-    </inertial>
-    <visual>
-      <origin rpy="0 0 0" xyz="0 0 0"/>
-      <geometry>
-        <mesh filename="$(arg path)/battery_2.STL"/>
-      </geometry>
-      <xacro:insert_block name="fiber"/>
-    </visual>
-  </link>
-  <joint name="battery_1_to_battery_2" type="fixed">
-    <origin rpy="0 0 0" xyz="0 -0.037 0"/>
-    <parent link="battery_1"/>
-    <child link="battery_2"/>
-    <axis xyz="0 0 0"/>
-  </joint>
-  <link name="mount">
-    <inertial>
-      <origin rpy="0 0 0" xyz="5.5511E-16 0.045908 -1.9984E-15"/>
-      <mass value="0.23261"/>
-      <inertia ixx="0" ixy="0" ixz="0" iyy="0" iyz="0" izz="0"/>
-    </inertial>
-    <visual>
-      <origin rpy="0 0 0" xyz="0 0 0"/>
-      <geometry>
-        <mesh filename="$(arg path)/mount.STL"/>
-      </geometry>
-      <xacro:insert_block name="fiber"/>
-    </visual>
-  </link>
-  <joint name="body_to_mount" type="fixed">
-    <origin rpy="1.5708 0 0" xyz="0.38768 -1.2531 0.56334"/>
-    <parent link="base_link"/>
-    <child link="mount"/>
-    <axis xyz="0 0 0"/>
-  </joint>
-  <link name="rs_232_port">
-    <inertial>
-      <origin rpy="0 0 0" xyz="6.911E-07 0.00015008 -0.0062931"/>
-      <mass value="0.0020002"/>
-      <inertia ixx="0" ixy="0" ixz="0" iyy="0" iyz="0" izz="0"/>
-    </inertial>
-    <visual>
-      <origin rpy="0 0 0" xyz="0 0 0"/>
-      <geometry>
-        <mesh filename="$(arg path)/rs_232_port.STL"/>
-      </geometry>
-      <xacro:insert_block name="fiber"/>
-    </visual>
-  </link>
-  <joint name="mount_to_port" type="fixed">
-    <origin rpy="-1.5708 0 0" xyz="0 0.0134 0.13225"/>
-    <parent link="mount"/>
-    <child link="rs_232_port"/>
-    <axis xyz="0 0 0"/>
-  </joint>
-  <link name="status_board">
-    <inertial>
-      <origin rpy="0 0 0" xyz="-0.00056781 0.0042824 0.02751"/>
-      <mass value="0.013407"/>
-      <inertia ixx="6.9707E-07" ixy="4.0982E-08" ixz="5.6997E-08" iyy="4.6531E-07" iyz="-3.2949E-07" izz="2.4594E-07"/>
-    </inertial>
-    <visual>
-      <origin rpy="0 0 0" xyz="0 0 0"/>
-      <geometry>
-        <mesh filename="$(arg path)/status_board.STL"/>
-      </geometry>
-      <xacro:insert_block name="fiber"/>
-    </visual>
-  </link>
-  <joint name="mount_to_status_board" type="fixed">
-    <origin rpy="0 0 0" xyz="-0.058 0.003 -0.032"/>
-    <parent link="mount"/>
-    <child link="status_board"/>
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