Commit message: Added new Model with fixed Mates

File: urdf/asv_base.xacro (robot description, xacro)
@@ -21,274 +21,402 @@
 	</joint>
 	<link name="base_link">
-		<inertial>
-			<origin rpy="0 0 0" xyz="0.00081248 -0.14905 0.79199"/>
-			<mass value="5.331"/>
-			<inertia ixx="0" ixy="0" ixz="0" iyy="0" iyz="0" izz="0"/>
-		</inertial>
-		<visual>
-			<origin rpy="0 0 0" xyz="0 0 0"/>
-			<geometry>
-				<mesh filename="$(arg path)/base_link.STL"/>
-			</geometry>
-			<xacro:insert_block name="fiber"/>
-		</visual>
-		<collision>
-			<origin rpy="0 0 0" xyz="0 0 0"/>
-			<geometry>
-				<mesh filename="$(arg path)/base_link.STL"/>
-			</geometry>
-		</collision>
-	</link>
-	<link name="thruster_left">
-		<inertial>
-			<origin rpy="0 0 0" xyz="-0.35951 -0.36784 0.94138"/>
-			<mass value="0.19486"/>
-			<inertia ixx="3.3635E-05" ixy="3.3962E-09" ixz="1.273E-07" iyy="3.3048E-05" iyz="-8.343E-07" izz="1.1884E-06"/>
-		</inertial>
-		<visual>
-			<origin rpy="0 0 0" xyz="0 0 0"/>
-			<geometry>
-				<mesh filename="$(arg path)/thruster_left.STL"/>
-			</geometry>
-			<xacro:insert_block name="fiber"/>
-		</visual>
-		<collision>
-			<origin rpy="0 0 0" xyz="0 0 0"/>
-			<geometry>
-				<mesh filename="$(arg path)/thruster_left.STL"/>
-			</geometry>
-		</collision>
-	</link>
-	<joint name="body_to_thruster_left" type="continuous">
-		<origin rpy="0 0 0" xyz="0 0 0"/>
-		<parent link="base_link"/>
-		<child link="thruster_left"/>
-		<axis xyz="0 0 0"/>
-		<!--<limit effort="30" lower="-32000" upper="32000" velocity="1.0"/>
-		<dynamics damping="0.1" friction="0.1"/>-->
-	</joint>
-	<link name="thruster_right">
-		<inertial>
-			<origin rpy="0 0 0" xyz="0.35962 -0.36784 0.94138"/>
-			<mass value="0.19487"/>
-			<inertia ixx="3.3633E-05" ixy="-8.3928E-09" ixz="-3.3111E-07" iyy="3.3048E-05" iyz="-8.3442E-07" izz="1.1913E-06"/>
-		</inertial>
-		<visual>
-			<origin rpy="0 0 0" xyz="0 0 0"/>
-			<geometry>
-				<mesh filename="$(arg path)/thruster_right.STL"/>
-			</geometry>
-			<material name="">
-				<color rgba="0.79216 0.81961 0.93333 1"/>
-			</material>
-		</visual>
-		<collision>
-			<origin rpy="0 0 0" xyz="0 0 0"/>
-			<geometry>
-				<mesh filename="$(arg path)/thruster_right.STL"/>
-			</geometry>
-		</collision>
-	</link>
-	<joint name="body_to_thruster_right" type="continuous">
-		<origin rpy="0 0 0" xyz="0 0 0"/>
-		<parent link="base_link"/>
-		<child link="thruster_right"/>
-		<axis xyz="0 0 0"/>
-		<!--<limit effort="30" lower="-32000" upper="32000" velocity="1.0"/>
-		<dynamics damping="0.1" friction="0.1"/>-->
-	</joint>
-	<link name="top_body">
-		<inertial>
-			<origin rpy="0 0 0" xyz="9.7484E-05 0.024673 0.7522"/>
-			<mass value="2.1573"/>
-			<inertia ixx="0.016871" ixy="-8.9301E-06" ixz="-3.158E-05" iyy="0.026678" iyz="-0.0021608" izz="0.010957"/>
-		</inertial>
-		<visual>
-			<origin rpy="0 0 0" xyz="0 0 0"/>
-			<geometry>
-				<mesh filename="$(arg path)/top_body.STL"/>
-			</geometry>
-			<xacro:insert_block name="fiber"/>
-		</visual>
-		<collision>
-			<origin rpy="0 0 0" xyz="0 0 0"/>
-			<geometry>
-				<mesh filename="$(arg path)/top_body.STL"/>
-			</geometry>
-		</collision>
-	</link>
-	<joint name="base_to_top" type="fixed">
-		<origin rpy="0 0 0" xyz="0 0 0"/>
-		<parent link="base_link"/>
-		<child link="top_body"/>
-		<axis xyz="0 0 0"/>
-	</joint>
-	<link name="sensor_pod">
-		<inertial>
-			<origin rpy="0 0 0" xyz="-0.013295 0.078554 0.22706"/>
-			<mass value="0.6495"/>
-			<inertia ixx="8.2722E-07" ixy="-6.7581E-06" ixz="3.6677E-05" iyy="0.0016822" iyz="1.4742E-07" izz="0.0016814"/>
-		</inertial>
-		<visual>
-			<origin rpy="0 0 0" xyz="0 0 0"/>
-			<geometry>
-				<mesh filename="$(arg path)/sensor_pod.STL"/>
-			</geometry>
-			<material name="">
-				<color rgba="0.79216 0.81961 0.93333 1"/>
-			</material>
-		</visual>
-		<collision>
-			<origin rpy="0 0 0" xyz="0 0 0"/>
-			<geometry>
-				<mesh filename="$(arg path)/sensor_pod.STL"/>
-			</geometry>
-		</collision>
-	</link>
-	<joint name="top_body_to_pod" type="fixed">
-		<origin rpy="0 0 0" xyz="0 0 0"/>
-		<parent link="top_body"/>
-		<child link="sensor_pod"/>
-		<axis xyz="0 0 0"/>
-	</joint>
-	<link name="lidar">
-		<inertial>
-			<origin rpy="0 0 0" xyz="0.007675 0.19969 0.070677"/>
-			<mass value="8.4876E-05"/>
-			<inertia ixx="7.4827E-08" ixy="1.2593E-09" ixz="-7.9614E-10" iyy="1.3889E-07" iyz="-1.1497E-08" izz="7.6608E-08"/>
-		</inertial>
-		<visual>
-			<origin rpy="0 0 0" xyz="0 0 0"/>
-			<geometry>
-				<mesh filename="$(arg path)/lidar.STL"/>
-			</geometry>
-			<material name="">
-				<color rgba="0.79216 0.81961 0.93333 1"/>
-			</material>
-		</visual>
-		<collision>
-			<origin rpy="0 0 0" xyz="0 0 0"/>
-			<geometry>
-				<mesh filename="$(arg path)/lidar.STL"/>
-			</geometry>
-		</collision>
-	</link>
-	<joint name="pod_to_lidar" type="continuous">
-		<origin rpy="0 0 0" xyz="0 0 0"/>
-		<parent link="sensor_pod"/>
-		<child link="lidar"/>
-		<axis xyz="1 0 0"/>
-	</joint>
-	<link name="camera_mount">
-		<inertial>
-			<origin rpy="0 0 0" xyz="-1.1102E-16 0.22615 0.20972"/>
-			<mass value="0.05273"/>
-			<inertia ixx="0" ixy="0" ixz="0" iyy="0" iyz="0" izz="0"/>
-		</inertial>
-		<visual>
-			<origin rpy="0 0 0" xyz="0 0 0"/>
-			<geometry>
-				<mesh filename="$(arg path)/camera_mount.STL"/>
-			</geometry>
-			<material name="">
-				<color rgba="1 1 1 0.875"/>
-			</material>
-		</visual>
-		<collision>
-			<origin rpy="0 0 0" xyz="0 0 0"/>
-			<geometry>
-				<mesh filename="$(arg path)/camera_mount.STL"/>
-			</geometry>
-		</collision>
-	</link>
-	<joint name="pod_to_camera_mount" type="fixed">
-		<origin rpy="0 0 0" xyz="0 0 0"/>
-		<parent link="sensor_pod"/>
-		<child link="camera_mount"/>
-		<axis xyz="0 0 0"/>
-	</joint>
-	<link name="camera">
-		<inertial>
-			<origin rpy="0 0 0" xyz="0.00010371 0.31918 0.16605"/>
-			<mass value="0.042277"/>
-			<inertia ixx="1.4944E-05" ixy="-4.7327E-08" ixz="5.3606E-08" iyy="3.1817E-06" iyz="3.9498E-06" izz="1.1765E-05"/>
-		</inertial>
-		<visual>
-			<origin rpy="0 0 0" xyz="0 0 0"/>
-			<geometry>
-				<mesh filename="$(arg path)/camera.STL"/>
-			</geometry>
-			<material name="">
-				<color rgba="0.019608 0.019608 0.019608 1"/>
-			</material>
-		</visual>
-		<collision>
-			<origin rpy="0 0 0" xyz="0 0 0"/>
-			<geometry>
-				<mesh filename="$(arg path)/camera.STL"/>
-			</geometry>
-		</collision>
-	</link>
-	<joint name="mount_to_camera" type="fixed">
-		<origin rpy="0 0 0" xyz="0 0 0"/>
-		<parent link="camera_mount"/>
-		<child link="camera"/>
-		<axis xyz="0 0 0"/>
-	</joint>
-	<link name="garmin_mount">
-		<inertial>
-			<origin rpy="0 0 0" xyz="-5.5511E-17 0.20372 0.27749"/>
-			<mass value="0.064841"/>
-			<inertia ixx="0" ixy="0" ixz="0" iyy="0" iyz="0" izz="0"/>
-		</inertial>
-		<visual>
-			<origin rpy="0 0 0" xyz="0 0 0"/>
-			<geometry>
-				<mesh filename="$(arg path)/garmin_mount.STL"/>
-			</geometry>
-			<material name="">
-				<color rgba="0.79216 0.81961 0.93333 1"/>
-			</material>
-		</visual>
-		<collision>
-			<origin rpy="0 0 0" xyz="0 0 0"/>
-			<geometry>
-				<mesh filename="$(arg path)/garmin_mount.STL"/>
-			</geometry>
-		</collision>
-	</link>
-	<joint name="pod_to_garmin_mount" type="fixed">
-		<origin rpy="0 0 0" xyz="0 0 0"/>
-		<parent link="sensor_pod"/>
-		<child link="garmin_mount"/>
-		<axis xyz="0 0 0"/>
-	</joint>
-	<link name="garmin">
-		<inertial>
-			<origin rpy="0 0 0" xyz="-1.1102E-16 0.23834 0.29679"/>
-			<mass value="0.3356"/>
-			<inertia ixx="0" ixy="0" ixz="0" iyy="0" iyz="0" izz="0"/>
-		</inertial>
-		<visual>
-			<origin rpy="0 0 0" xyz="0 0 0"/>
-			<geometry>
-				<mesh filename="$(arg path)/garmin.STL"/>
-			</geometry>
-			<material name="">
-				<color rgba="0.79216 0.81961 0.93333 1"/>
-			</material>
-		</visual>
-		<collision>
-			<origin rpy="0 0 0" xyz="0 0 0"/>
-			<geometry>
-				<mesh filename="$(arg path)/garmin.STL"/>
-			</geometry>
-		</collision>
-	</link>
-	<joint name="gps_to_mount" type="fixed">
-		<origin rpy="0 0 0" xyz="0 0 0"/>
-		<parent link="garmin_mount"/>
-		<child link="garmin"/>
-		<axis xyz="0 0 0"/>
-	</joint>
+    <inertial>
+      <origin rpy="0 0 0" xyz="0.00081244 -0.14905 0.79199"/>
+      <mass value="5.331"/>
+      <inertia ixx="0" ixy="0" ixz="0" iyy="0" iyz="0" izz="0"/>
+    </inertial>
+    <visual>
+      <origin rpy="0 0 0" xyz="0 0 0"/>
+      <geometry>
+        <mesh filename="$(arg path)/base_link.STL"/>
+      </geometry>
+      <material name="">
+        <color rgba="0.79216 0.81961 0.93333 1"/>
+      </material>
+    </visual>
+    <collision>
+      <origin rpy="0 0 0" xyz="0 0 0"/>
+      <geometry>
+        <mesh filename="$(arg path)/base_link.STL"/>
+      </geometry>
+    </collision>
+  </link>
+  <link name="thruster_left">
+    <inertial>
+      <origin rpy="0 0 0" xyz="-5.8627E-05 0.00058333 0.0038275"/>
+      <mass value="0.18712"/>
+      <inertia ixx="3.3531E-05" ixy="2.291E-09" ixz="-1.0217E-07" iyy="3.2946E-05" iyz="8.185E-07" izz="1.1857E-06"/>
+    </inertial>
+    <visual>
+      <origin rpy="0 0 0" xyz="0 0 0"/>
+      <geometry>
+        <mesh filename="$(arg path)/thruster_left.STL"/>
+      </geometry>
+      <material name="">
+        <color rgba="0.79216 0.81961 0.93333 1"/>
+      </material>
+    </visual>
+    <collision>
+      <origin rpy="0 0 0" xyz="0 0 0"/>
+      <geometry>
+        <mesh filename="$(arg path)/thruster_left.STL"/>
+      </geometry>
+    </collision>
+  </link>
+  <joint name="body_to_thruster_left" type="fixed">
+    <origin rpy="3.1416 -0.034204 -3.1416" xyz="-0.36527 -0.3684 0.94656"/>
+    <parent link="base_link"/>
+    <child link="thruster_left"/>
+    <axis xyz="0 0 0"/>
+  </joint>
+  <link name="left_prop">
+    <inertial>
+      <origin rpy="0 0 0" xyz="-8.9802E-06 -7.9168E-05 1.1483E-06"/>
+      <mass value="0.0055557"/>
+      <inertia ixx="3.8077E-07" ixy="-2.1107E-10" ixz="-7.6917E-11" iyy="7.603E-07" iyz="2.5415E-11" izz="3.798E-07"/>
+    </inertial>
+    <visual>
+      <origin rpy="0 0 0" xyz="0 0 0"/>
+      <geometry>
+        <mesh filename="$(arg path)/left_prop.STL"/>
+      </geometry>
+      <material name="">
+        <color rgba="0.79216 0.81961 0.93333 1"/>
+      </material>
+    </visual>
+    <collision>
+      <origin rpy="0 0 0" xyz="0 0 0"/>
+      <geometry>
+        <mesh filename="$(arg path)/left_prop.STL"/>
+      </geometry>
+    </collision>
+  </link>
+  <joint name="left_thruster_to_prop" type="continuous">
+    <origin rpy="-1.5708 -1.1015E-15 -1.8579" xyz="0 0 0.0101"/>
+    <parent link="thruster_left"/>
+    <child link="left_prop"/>
+    <axis xyz="0 0 0"/>
+    <limit effort="0.098067" velocity="397.94"/>
+  </joint>
+  <link name="thruster_right">
+    <inertial>
+      <origin rpy="0 0 0" xyz="-5.8645E-05 0.00058315 0.0038281"/>
+      <mass value="0.18712"/>
+      <inertia ixx="3.3529E-05" ixy="2.2892E-09" ixz="-1.0218E-07" iyy="3.2945E-05" iyz="8.1817E-07" izz="1.1857E-06"/>
+    </inertial>
+    <visual>
+      <origin rpy="0 0 0" xyz="0 0 0"/>
+      <geometry>
+        <mesh filename="$(arg path)/thruster_right.STL"/>
+      </geometry>
+      <material name="">
+        <color rgba="0.79216 0.81961 0.93333 1"/>
+      </material>
+    </visual>
+    <collision>
+      <origin rpy="0 0 0" xyz="0 0 0"/>
+      <geometry>
+        <mesh filename="$(arg path)/thruster_right.STL"/>
+      </geometry>
+    </collision>
+  </link>
+  <joint name="body_to_thruster_right" type="fixed">
+    <origin rpy="3.1416 0.034204 3.1416" xyz="0.36311 -0.3684 0.94648"/>
+    <parent link="base_link"/>
+    <child link="thruster_right"/>
+    <axis xyz="0 0 0"/>
+  </joint>
+  <link name="right_prop">
+    <inertial>
+      <origin rpy="0 0 0" xyz="-2.86418217365636E-07 -7.95554534813725E-05 -9.67893664827191E-07"/>
+      <mass value="0.00555700041550943"/>
+      <inertia ixx="3.80620473025844E-07" ixy="-1.02454560847702E-11" ixz="-1.5511326553023E-11" iyy="7.6093135544076E-07" iyz="-4.82655749375765E-11" izz="3.80581124486253E-07"/>
+    </inertial>
+    <visual>
+      <origin rpy="0 0 0" xyz="0 0 0"/>
+      <geometry>
+        <mesh filename="$(arg path)/right_prop.STL"/>
+      </geometry>
+			<xacro:insert_block name="fiber"/>
+    </visual>
+    <collision>
+      <origin rpy="0 0 0" xyz="0 0 0"/>
+      <geometry>
+        <mesh filename="$(arg path)/right_prop.STL"/>
+      </geometry>
+    </collision>
+  </link>
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
Commit message: Calibration Level 1

File: urdf/asv_base.xacro (robot description, xacro)
@@ -93,5 +93,5 @@
   </link>
   <joint name="left_thruster_to_prop" type="continuous">
-    <origin rpy="-1.5708 -1.1015E-15 -1.8579" xyz="0 0 0.0101"/>
+    <origin rpy="-1.5708 0 -1.8579" xyz="0 0 0.0101"/>
     <parent link="thruster_left"/>
     <child link="left_prop"/>

Commit message: Modified the props for better Mates

File: urdf/asv_base.xacro (robot description, xacro)
@@ -42,9 +42,9 @@
     </collision>
   </link>
-  <link name="thruster_left">
-    <inertial>
-      <origin rpy="0 0 0" xyz="-5.8627E-05 0.00058333 0.0038275"/>
-      <mass value="0.18712"/>
-      <inertia ixx="3.3531E-05" ixy="2.291E-09" ixz="-1.0217E-07" iyy="3.2946E-05" iyz="8.185E-07" izz="1.1857E-06"/>
+<link name="thruster_left">
+    <inertial>
+      <origin rpy="0 0 0" xyz="0.00850178534589952 0.0511449724847095 -5.42946450400594E-05"/>
+      <mass value="0.201295638408416"/>
+      <inertia ixx="3.60508026375113E-05" ixy="-6.37790577446859E-06" ixz="-9.55155846597797E-08" iyy="3.38328251838062E-05" iyz="3.94192413473368E-08" izz="6.92827790100947E-05"/>
     </inertial>
     <visual>
@@ -53,7 +53,5 @@
         <mesh filename="$(arg path)/thruster_left.STL"/>
       </geometry>
-      <material name="">
-        <color rgba="0.79216 0.81961 0.93333 1"/>
-      </material>
+      <xacro:insert_block name="fiber"/>
     </visual>
     <collision>
@@ -65,5 +63,5 @@
   </link>
   <joint name="body_to_thruster_left" type="fixed">
-    <origin rpy="3.1416 -0.034204 -3.1416" xyz="-0.36527 -0.3684 0.94656"/>
+    <origin rpy="0 1.5366 3.1416" xyz="-0.36509 -0.31305 0.95181"/>
     <parent link="base_link"/>
     <child link="thruster_left"/>
@@ -99,9 +97,9 @@
     <limit effort="0.098067" velocity="397.94"/>
   </joint>
-  <link name="thruster_right">
-    <inertial>
-      <origin rpy="0 0 0" xyz="-5.8645E-05 0.00058315 0.0038281"/>
-      <mass value="0.18712"/>
-      <inertia ixx="3.3529E-05" ixy="2.2892E-09" ixz="-1.0218E-07" iyy="3.2945E-05" iyz="8.1817E-07" izz="1.1857E-06"/>
+    <link name="thruster_right">
+    <inertial>
+      <origin rpy="0 0 0" xyz="0.00850255972055614 0.051144652615246 -5.43497983066521E-05"/>
+      <mass value="0.201292014430916"/>
+      <inertia ixx="3.60548334017782E-05" ixy="-6.37582458259697E-06" ixz="-9.55850176393278E-08" iyy="3.38303930900005E-05" iyz="3.90578037394754E-08" izz="6.92844408354745E-05"/>
     </inertial>
     <visual>
@@ -110,7 +108,5 @@
         <mesh filename="$(arg path)/thruster_right.STL"/>
       </geometry>
-      <material name="">
-        <color rgba="0.79216 0.81961 0.93333 1"/>
-      </material>
+      <xacro:insert_block name="fiber"/>
     </visual>
     <collision>
@@ -122,5 +118,5 @@
   </link>
   <joint name="body_to_thruster_right" type="fixed">
-    <origin rpy="3.1416 0.034204 3.1416" xyz="0.36311 -0.3684 0.94648"/>
+    <origin rpy="3.1416 1.5366 0" xyz="0.36293 -0.31305 0.95173"/>
     <parent link="base_link"/>
     <child link="thruster_right"/>

Commit message: Stashing changes for further use

File: urdf/asv_base.xacro (robot description, xacro)
@@ -71,5 +71,5 @@
     <inertial>
       <origin rpy="0 0 0" xyz="-8.9802E-06 -7.9168E-05 1.1483E-06"/>
-      <mass value="0.0055557"/>
+      <mass value="0.125"/>
       <inertia ixx="3.8077E-07" ixy="-2.1107E-10" ixz="-7.6917E-11" iyy="7.603E-07" iyz="2.5415E-11" izz="3.798E-07"/>
     </inertial>
@@ -126,5 +126,5 @@
     <inertial>
       <origin rpy="0 0 0" xyz="-2.86418217365636E-07 -7.95554534813725E-05 -9.67893664827191E-07"/>
-      <mass value="0.00555700041550943"/>
+      <mass value="0.125"/>
       <inertia ixx="3.80620473025844E-07" ixy="-1.02454560847702E-11" ixz="-1.5511326553023E-11" iyy="7.6093135544076E-07" iyz="-4.82655749375765E-11" izz="3.80581124486253E-07"/>
     </inertial>
@@ -303,5 +303,5 @@
     </collision>
   </link>
-  <joint name="pod_to_lidar" type="revolute">
+  <joint name="pod_to_lidar" type="fixed">
     <origin rpy="0 -1.5706 1.9266" xyz="0.096667 0.046463 -0.0605"/>
     <parent link="sensor_pod"/>

Commit message: Final changes stashed

File: urdf/asv_base.xacro (robot description, xacro)
@@ -1,4 +1,5 @@
 <?xml version="1.0"?>
 <robot name="asv_description" xmlns:xacro="http://www.ros.org/wiki/xacro">
+  <xacro:include filename="$(find asv_description)/urdf/common_properties.xacro"/>
   <link name="base_footprint">
     <inertial>
@@ -15,5 +16,5 @@
   </link>
   <joint name="base_footprint_joint" type="fixed">
-    <origin rpy="0 0 0" xyz="0 0 0"/>
+    <origin rpy="0 0 -${PI/2}" xyz="0 0 0"/>
     <parent link="base_footprint"/>
     <child link="base_link"/>
@@ -65,5 +66,5 @@
     </collision>
   </link>
-  <joint name="body_to_thruster_right" type="continuous">
+  <joint name="body_to_thruster_right" type="fixed">
     <origin rpy="1.5708 0 3.1416" xyz="0.74762 -1.335 0.37124"/>
     <parent link="thruster_right_dummy"/>
@@ -105,5 +106,5 @@
     </collision>
   </link>
-  <joint name="body_to_thruster_left" type="continuous">
+  <joint name="body_to_thruster_left" type="fixed">
     <origin rpy="1.5708 0 3.1416" xyz="0.027678 -1.335 0.37124"/>
     <parent link="thruster_left_dummy"/>
@@ -161,5 +162,5 @@
     <inertial>
       <origin rpy="0 0 0" xyz="-0.029193 -0.040604 -0.010551"/>
-      <mass value="0.06495"/>
+      <mass value="0.6495"/>
       <inertia ixx="0.0016814" ixy="-1.4742E-07" ixz="-3.6677E-05" iyy="0.0016822" iyz="-6.7581E-06" izz="8.2722E-07"/>
     </inertial>
@@ -181,5 +182,5 @@
     <inertial>
       <origin rpy="0 0 0" xyz="0.0027436 0.024777 0.009305"/>
-      <mass value="0.011757"/>
+      <mass value="0.11757"/>
       <inertia ixx="0.0001482" ixy="1.0861E-19" ixz="-3.2822E-19" iyy="0.00013357" iyz="4.4199E-05" izz="1.4626E-05"/>
     </inertial>
@@ -201,5 +202,5 @@
     <inertial>
       <origin rpy="3.141592653589793 0 0" xyz="0 0.023342 0"/>
-      <mass value="0.03356"/>
+      <mass value="0.3356"/>
       <inertia ixx="0" ixy="0" ixz="0" iyy="0" iyz="0" izz="0"/>
     </inertial>
@@ -221,5 +222,5 @@
     <inertial>
       <origin rpy="0 0 0" xyz="-2.8934E-05 -0.010178 0.021487"/>
-      <mass value="0.0041091"/>
+      <mass value="0.041091"/>
       <inertia ixx="1.4847E-05" ixy="-3.2519E-08" ixz="-1.1631E-08" iyy="3.365E-06" iyz="-4.1204E-06" izz="1.1483E-05"/>
     </inertial>
@@ -263,5 +264,5 @@
     <inertial>
       <origin rpy="0 0 0" xyz="0.21906 0.04363 0.013308"/>
-      <mass value="0.0048397"/>
+      <mass value="0.048397"/>
       <inertia ixx="0" ixy="0" ixz="0" iyy="0" iyz="0" izz="0"/>
     </inertial>
@@ -283,5 +284,5 @@
     <inertial>
       <origin rpy="0 0 0" xyz="0.21906 0.04363 0.013308"/>
-      <mass value="0.0048397"/>
+      <mass value="0.048397"/>
       <inertia ixx="0" ixy="0" ixz="0" iyy="0" iyz="0" izz="0"/>
     </inertial>
@@ -363,5 +364,5 @@
     <inertial>
       <origin rpy="0 0 0" xyz="6.911E-07 0.00015008 -0.0062931"/>
-      <mass value="0.0020002"/>
+      <mass value="0.020002"/>
       <inertia ixx="0" ixy="0" ixz="0" iyy="0" iyz="0" izz="0"/>
     </inertial>
@@ -383,5 +384,5 @@
     <inertial>
       <origin rpy="0 0 0" xyz="-0.00056781 0.0042824 0.02751"/>
-      <mass value="0.013407"/>
+      <mass value="0.13407"/>
       <inertia ixx="6.9707E-07" ixy="4.0982E-08" ixz="5.6997E-08" iyy="4.6531E-07" iyz="-3.2949E-07" izz="2.4594E-07"/>
     </inertial>

Commit message: New lidar model from the lms1xx plugin

File: urdf/asv_base.xacro (robot description, xacro)
@@ -250,5 +250,5 @@
       <origin rpy="0 0 0" xyz="0 0 0"/>
       <geometry>
-        <mesh filename="$(arg path)/lidar.STL"/>
+        <mesh filename="package://lms1xx/meshes/sick-lms1xx.dae"/>
       </geometry>
       <xacro:insert_block name="fiber"/>
