Commit message: Stashing commits before modifying local system

File: urdf/asv_base.xacro (robot description, xacro)
@@ -1,27 +1,22 @@
 <?xml version="1.0"?>
 <robot name="asv_description" xmlns:xacro="http://www.ros.org/wiki/xacro">
-  <xacro:include filename="$(find asv_description)/urdf/common_properties.xacro"/>
-  <link name="base_footprint">
-    <inertial>
-      <mass value="0.0001"/>
-      <origin xyz="0 0 0" rpy="0 0 0"/>
-      <inertia ixx="0.0001" ixy="0.0" ixz="0.0" iyy="0.0001" iyz="0.0" izz="0.0001"/>
-    </inertial>
-    <visual>
-      <origin rpy="0 0 0" xyz="0 0 0"/>
-      <geometry>
-        <box size="0.001 0.001 0.001"/>
-      </geometry>
-    </visual>
-  </link>
-  <joint name="base_footprint_joint" type="fixed">
-    <origin rpy="${PI/2} 0 ${-PI/2}" xyz="0 0 0.75"/>
-    <parent link="base_footprint"/>
-    <child link="base_link"/>
-  </joint>
   <link name="base_link">
-    <inertial>
-      <origin rpy="0 0 0" xyz="0 0 0"/>
-      <mass value="8.3305"/>
+    <collision>
+      <origin rpy="0 0 0" xyz="0 0 0"/>
+      <geometry>
+        <box size="5 5 0.4" />
+      </geometry>
+      <!--<contact_coefficients mu="0.1" kp="0.2" kd="0.5" />-->
+    </collision>
+  </link>
+  <joint name="virtual_joint" type="fixed">
+    <origin xyz="0 0 2" rpy="0 0 0" />
+    <parent link="base_link"/>
+    <child link="base_hull"/>
+  </joint>
+  <link name="base_hull">
+    <inertial>
+      <origin rpy="0 0 0" xyz="0 0 0"/>
+      <mass value="20.3305"/>
       <inertia ixx="0.48818" ixy="-1.0031E-06" ixz="-0.00052597" iyy="0.77995" iyz="0.060345" izz="0.40032"/>
     </inertial>
@@ -29,5 +24,5 @@
       <origin rpy="0 0 0" xyz="0 0 0"/>
       <geometry>
-        <mesh filename="package://asv_description/meshes/base_link.STL"/>
+        <mesh filename="package://asv_description/meshes/base_link.dae"/>
       </geometry>
       <xacro:insert_block name="fiber"/>
@@ -36,9 +31,11 @@
       <origin rpy="0 0 0" xyz="0 0 0"/>
       <geometry>
-        <mesh filename="package://asv_description/meshes/base_link.STL"/>
-      </geometry>
+        <mesh filename="package://asv_description/meshes/base_link.dae"/>
+        <!--<box size="0.1 0.1 0.1" />-->
+      </geometry>
+      <!--<contact_coefficients mu="0.1" kp="0.2" kd="0.5" />-->
     </collision>
   </link>
-  <link name="thruster_left">
+  <!--<link name="thruster_left">
     <inertial>
       <origin xyz="-5.6771E-05 0.0040313 0.0046012" rpy="0 0 0" />
@@ -53,14 +50,8 @@
       <xacro:insert_block name="fiber"/>
     </visual>
-    <collision>
-      <origin rpy="0 0 0" xyz="0 0 0"/>
-      <geometry>
-        <mesh filename="package://asv_description/meshes/thruster_left.STL"/>
-      </geometry>
-    </collision>
   </link>
   <joint name="body_to_thruster_left" type="fixed">
     <origin xyz="-0.36142 -0.26516 0.17933" rpy="0.13754 -0.00034105 -4.7207E-05" />
-    <parent link="base_link"/>
+    <parent link="base_hull"/>
     <child link="thruster_left"/>
     <axis xyz="0 0 0"/>
@@ -79,14 +70,8 @@
       <xacro:insert_block name="fiber"/>
     </visual>
-    <collision>
-      <origin rpy="0 0 0" xyz="0 0 0"/>
-      <geometry>
-        <mesh filename="package://asv_description/meshes/thruster_right.STL" />
-      </geometry>
-    </collision>
   </link>
   <joint name="body_to_thruster_right" type="fixed">
     <origin xyz="0.36046 -0.21222 0.20053" rpy="-1.5683 1.4333 1.5733" />
-    <parent link="base_link"/>
+    <parent link="base_hull"/>
     <child link="thruster_right"/>
     <axis xyz="0 0 0"/>
@@ -105,14 +90,8 @@
       <xacro:insert_block name="fiber"/>
     </visual>
-    <collision>
-      <origin xyz="0 0 0" rpy="0 0 0" />
-      <geometry>
-        <mesh filename="package://asv_description/meshes/top_body.STL" />
-      </geometry>
-    </collision>
   </link>
   <joint name="base_to_top_body" type="fixed">
     <origin xyz="-0.00047785 0.0019807 -0.052277" rpy="0.13754 0 0" />
-    <parent link="base_link" />
+    <parent link="base_hull" />
     <child link="top_body" />
     <axis xyz="0 0 0" />
@@ -131,10 +110,4 @@
       <xacro:insert_block name="fiber"/>
     </visual>
-    <collision>
-      <origin xyz="0 0 0" rpy="0 0 0" />
-      <geometry>
-        <mesh filename="package://asv_description/meshes/top_cover.STL" />
-      </geometry>
-    </collision>
   </link>
   <joint name="top_body_to_cover" type="fixed">
@@ -159,10 +132,4 @@
       </material>
     </visual>
-    <collision>
-      <origin xyz="0 0 0" rpy="0 0 0" />
-      <geometry>
-        <mesh filename="package://asv_description/meshes/sensor_pod.STL" />
-      </geometry>
-    </collision>
   </link>
     <joint name="top_to_sensor_pod" type="fixed">
@@ -183,14 +150,8 @@
         <origin xyz="0 0 0" rpy="0 0 0" />
         <geometry>
-          <!-- Origin of this mesh is the focal point of the LIDAR. -->
-          <mesh filename="package://lms1xx/meshes/sick-lms1xx.dae" />
+          <! Origin of this mesh is the focal point of the LIDAR. -->
+          <!--<mesh filename="package://lms1xx/meshes/sick-lms1xx.dae" />
         </geometry>
       </visual>
-      <collision>
-        <origin xyz="0 0 -0.05" rpy="0 0 0" />
-        <geometry>
-          <box size="0.105 0.1 0.1" />
-        </geometry>
-      </collision>
   </link>
   <joint name="pod_to_lidar" type="fixed">
@@ -215,10 +176,4 @@
       </material>
     </visual>
-    <collision>
-      <origin xyz="0 0 0" rpy="0 0 0" />
-      <geometry>
-        <mesh filename="package://asv_description/meshes/garmin.STL" />
-      </geometry>
-    </collision>
   </link>
   <joint name="top_to_garmin" type="fixed">
@@ -243,10 +198,4 @@
       </material>
     </visual>
-    <collision>
-      <origin xyz="0 0 0" rpy="0 0 0" />
-      <geometry>
-        <mesh filename="package://asv_description/meshes/camera.STL" />
-      </geometry>
-    </collision>
   </link>
   <joint name="pod_to_camera" type="fixed">
@@ -271,14 +220,8 @@
       </material>
     </visual>
-    <collision>
-      <origin xyz="0 0 0" rpy="0 0 0" />
-      <geometry>
-        <mesh filename="package://asv_description/meshes/middle_hull.STL" />
-      </geometry>
-    </collision>
   </link>
   <joint name="base_to_middle_hull" type="fixed">
     <origin xyz="0.0001217 -0.038509 -0.098623" rpy="0.13754 0 0" />
-    <parent link="base_link" />
+    <parent link="base_hull" />
     <child link="middle_hull" />
     <axis xyz="0 0 0" />
@@ -299,10 +242,4 @@
       </material>
     </visual>
-    <collision>
-      <origin xyz="0 0 0" rpy="0 0 0" />
-      <geometry>
-        <mesh filename="package://asv_description/meshes/mount.STL" />
-      </geometry>
-    </collision>
   </link>
   <joint name="hull_to_mount" type="fixed">
@@ -327,10 +264,4 @@
       </material>
     </visual>
-    <collision>
-      <origin xyz="0 0 0" rpy="0 0 0" />
-      <geometry>
-        <mesh filename="package://asv_description/meshes/electronics.STL" />
-      </geometry>
-    </collision>
   </link>
   <joint name="mount_electronics" type="fixed">
@@ -355,10 +286,4 @@
       </material>
     </visual>
-    <collision>
-      <origin xyz="0 0 0" rpy="0 0 0" />
-      <geometry>
-        <mesh filename="package://asv_description/meshes/rs232.STL" />
-      </geometry>
-    </collision>
   </link>
   <joint name="mount_to_rs232" type="fixed">
@@ -383,10 +308,4 @@
       </material>
     </visual>
-    <collision>
-      <origin xyz="0 0 0" rpy="0 0 0" />
-      <geometry>
-        <mesh filename="package://asv_description/meshes/battery_1.STL" />
-      </geometry>
-    </collision>
   </link>
   <joint name="hull_to_battery_1" type="fixed">
@@ -411,10 +330,4 @@
       </material>
     </visual>
-    <collision>
-      <origin xyz="0 0 0" rpy="0 0 0" />
-      <geometry>
-        <mesh filename="package://asv_description/meshes/battery_2.STL" />
-      </geometry>
-    </collision>
   </link>
   <joint name="hull_to_battery_2" type="fixed">
@@ -423,4 +336,4 @@
     <child link="battery_2" />
     <axis xyz="0 0 0" />
-  </joint>
+  </joint>-->
 </robot>
